Commit message: First commit - Fixed issued with hand control in moveit

File: panda_softhand_moveit_config/config/hand.xacro (robot description, xacro)
@@ -1,23 +1,37 @@
-<?xml version="1.0" ?>
-<robot xmlns:xacro="http://www.ros.org/wiki/xacro" name="panda">
-  <xacro:macro name="hand">
-    <!--GROUPS: Representation of a set of joints and links. This can be useful for specifying DOF to plan for, defining arms, end effectors, etc-->
-    <!--LINKS: When a link is specified, the parent joint of that link (if it exists) is automatically included-->
-    <!--JOINTS: When a joint is specified, the child link of that joint (which will always exist) is automatically included-->
-    <!--CHAINS: When a chain is specified, all the links along the chain (including endpoints) are included in the group. Additionally, all the joints that are parents to included links are also included. This means that joints along the chain and the parent joint of the base link are included in the group-->
-    <!--SUBGROUPS: Groups can also be formed by referencing to already defined group names-->
-    <group name="hand">
-      <link name="panda_hand" />
-      <link name="panda_leftfinger" />
-      <link name="panda_rightfinger" />
-      <joint name="panda_finger_joint1" />
-      <passive_joint name="panda_finger_joint2" />
-    </group>
-    <!--GROUP STATES: Purpose: Define a named state for a particular group, in terms of joint values. This is useful to define states like 'folded arms'-->
-    <!--END EFFECTOR: Purpose: Represent information about an end effector.-->
-    <!--DISABLE COLLISIONS: By default it is assumed that any link of the robot could potentially come into collision with any other link in the robot. This tag disables collision checking between a specified pair of links. -->
-    <disable_collisions link1="panda_hand" link2="panda_leftfinger" reason="Adjacent" />
-    <disable_collisions link1="panda_hand" link2="panda_rightfinger" reason="Adjacent" />
-    <disable_collisions link1="panda_leftfinger" link2="panda_rightfinger" reason="Default" />
-  </xacro:macro>
+<?xml version="1.0" encoding="UTF-8"?>
+<robot xmlns:xacro="http://www.ros.org/wiki/xacro" name="right">
+    <xacro:macro name="hand">
+        <!--GROUPS: Representation of a set of joints and links. This can be useful for specifying DOF to plan for, defining arms, end effectors, etc-->
+        <!--LINKS: When a link is specified, the parent joint of that link (if it exists) is automatically included-->
+        <!--JOINTS: When a joint is specified, the child link of that joint (which will always exist) is automatically included-->
+        <!--CHAINS: When a chain is specified, all the links along the chain (including endpoints) are included in the group. Additionally, all the joints that are parents to included links are also included. This means that joints along the chain and the parent joint of the base link are included in the group-->
+        <!--SUBGROUPS: Groups can also be formed by referencing to already defined group names-->
+        <group name="right_hand">
+            <joint name="right_hand_synergy_joint"/>
+        </group>
+        <!--GROUP STATES: Purpose: Define a named state for a particular group, in terms of joint values. This is useful to define states like 'folded arms'-->
+        <group_state name="open" group="right_hand">
+            <joint name="right_hand_synergy_joint" value="0.0"/>
+        </group_state>
+        <group_state name="close" group="right_hand">
+            <joint name="right_hand_synergy_joint" value="0.9"/>
+        </group_state>
+        <!--END EFFECTOR: Purpose: Represent information about an end effector.-->
+        <!--VIRTUAL JOINT: Purpose: this element defines a virtual joint between a robot link and an external frame of reference (considered fixed with respect to the robot)-->
+        <!--PASSIVE JOINT: Purpose: this element is used to mark joints that are not actuated-->
+        <!--DISABLE COLLISIONS: By default it is assumed that any link of the robot could potentially come into collision with any other link in the robot. This tag disables collision checking between a specified pair of links. -->
+        <!-- Disable collisions for hand_sc by default (with environment) -->
+        <!-- <disable_default_collisions link="$(arg arm_id)_hand" /> -->
+        <!-- Reenable collision of hand_sc for selected arm sc links -->
+        <!-- <xacro:property name="link_fmt" value="$(arg arm_id)_link{}" /> -->
+        <!-- <xacro:enable_collisions_for link="$(arg arm_id)_hand_sc" others="${[link_fmt.format(i) for i in [0,1,2,3]]}" /> -->
+        <!-- Disable collision of hand link with all arm links. These are handled by the *_sc links -->
+        <!-- <xacro:property name="link_fmt" value="$(arg arm_id)_link{}" />
+        <xacro:disable_collisions_for link="$(arg arm_id)_hand" others="${[link_fmt.format(i) for i in python.range(8)]}" /> -->
+        <!-- Disable collision of fingers with all arm links -->
+        <!-- <xacro:property name="others" value="${[link_fmt.format(i) for i in python.range(8)] + [xacro.arg('arm_id') + '_hand']}" />
+        <xacro:disable_collisions_for link="$(arg arm_id)_leftfinger" others="${list(others)}" />
+        <xacro:disable_collisions_for link="$(arg arm_id)_rightfinger" others="${list(others)}" />
+        <disable_collisions link1="$(arg arm_id)_leftfinger" link2="$(arg arm_id)_rightfinger" reason="Never" /> -->
+    </xacro:macro>
 </robot>

File: panda_softhand_moveit_config/config/panda_arm.xacro (robot description, xacro)
@@ -44,4 +44,6 @@
     <disable_collisions link1="panda_link5" link2="panda_link6" reason="Adjacent" />
     <disable_collisions link1="panda_link6" link2="panda_link7" reason="Adjacent" />
+    <disable_collisions link1="panda_link8" link2="right_hand_panda_flange" reason="Adjacent" />
+    <disable_collisions link1="panda_link7" link2="panda_link8" reason="Adjacent" />
     <!--ADDITIONALLY ADDED-->
     <passive_joint name="right_hand_index_abd_joint" />

File: panda_softhand_moveit_config/config/panda_arm_hand.srdf.xacro (robot description, xacro)
@@ -5,6 +5,6 @@
 -->
 <robot xmlns:xacro="http://www.ros.org/wiki/xacro" name="panda">
-  <xacro:include filename="$(find panda_moveit_config)/config/panda_arm.xacro" />
-  <xacro:include filename="$(find panda_moveit_config)/config/hand.xacro" />
+  <xacro:include filename="$(find panda_softhand_moveit_config)/config/panda_arm.xacro" />
+  <xacro:include filename="$(find panda_softhand_moveit_config)/config/hand.xacro" />
   <xacro:panda_arm />
   <xacro:hand />
@@ -16,5 +16,5 @@
   <group name="panda_arm_hand">
     <group name="panda_arm" />
-    <group name="hand" />
+    <group name="right_hand" />
   </group>
   <!--GROUP STATES: Purpose: Define a named state for a particular group, in terms of joint values. This is useful to define states like 'folded arms'-->
@@ -27,19 +27,8 @@
     <joint name="panda_joint6" value="1.571" />
     <joint name="panda_joint7" value="0.785" />
+    <joint name="right_hand_synergy_joint" value="0.0" />
   </group_state>
   <!--END EFFECTOR: Purpose: Represent information about an end effector.-->
-  <end_effector name="hand" parent_link="panda_link8" group="hand" parent_group="panda_arm" />
+  <!-- <end_effector name="hand" parent_link="panda_link8" group="hand" parent_group="panda_arm" /> -->
   <!--DISABLE COLLISIONS: By default it is assumed that any link of the robot could potentially come into collision with any other link in the robot. This tag disables collision checking between a specified pair of links. -->
-  <disable_collisions link1="panda_hand" link2="panda_link3" reason="Never" />
-  <disable_collisions link1="panda_hand" link2="panda_link4" reason="Never" />
-  <disable_collisions link1="panda_hand" link2="panda_link6" reason="Never" />
-  <disable_collisions link1="panda_hand" link2="panda_link7" reason="Adjacent" />
-  <disable_collisions link1="panda_leftfinger" link2="panda_link3" reason="Never" />
-  <disable_collisions link1="panda_leftfinger" link2="panda_link4" reason="Never" />
-  <disable_collisions link1="panda_leftfinger" link2="panda_link6" reason="Never" />
-  <disable_collisions link1="panda_leftfinger" link2="panda_link7" reason="Never" />
-  <disable_collisions link1="panda_link3" link2="panda_rightfinger" reason="Never" />
-  <disable_collisions link1="panda_link4" link2="panda_rightfinger" reason="Never" />
-  <disable_collisions link1="panda_link6" link2="panda_rightfinger" reason="Never" />
-  <disable_collisions link1="panda_link7" link2="panda_rightfinger" reason="Never" />
 </robot>
