Commit message: Added description and solved build issues.

File: panda_softhand_moveit_config/config/gazebo_panda_softhand.urdf (robot description, URDF)
Before this commit: robot panda_softhand, 51 links, 50 joints
Links:
- removed link qbhand2m1_90_deg_flange_base_link
- removed link qbhand2m1_base_link
- removed link qbhand2m1_index_distal_link
- removed link qbhand2m1_index_distal_virtual_link
- removed link qbhand2m1_index_knuckle_link
- removed link qbhand2m1_index_middle_link
- removed link qbhand2m1_index_middle_virtual_link
- removed link qbhand2m1_index_proximal_link
- removed link qbhand2m1_index_proximal_virtual_link
- removed link qbhand2m1_little_distal_link
- removed link qbhand2m1_little_distal_virtual_link
- removed link qbhand2m1_little_knuckle_link
- removed link qbhand2m1_little_middle_link
- removed link qbhand2m1_little_middle_virtual_link
- removed link qbhand2m1_little_proximal_link
- removed link qbhand2m1_little_proximal_virtual_link
- removed link qbhand2m1_manipulation_tendon_virtual_link
- removed link qbhand2m1_middle_distal_link
- removed link qbhand2m1_middle_distal_virtual_link
- removed link qbhand2m1_middle_knuckle_link
- removed link qbhand2m1_middle_middle_link
- removed link qbhand2m1_middle_middle_virtual_link
- removed link qbhand2m1_middle_proximal_link
- removed link qbhand2m1_middle_proximal_virtual_link
- removed link qbhand2m1_motor_1_tendon_virtual_link
- removed link qbhand2m1_motor_2_tendon_virtual_link
- removed link qbhand2m1_palm_link
- removed link qbhand2m1_ring_distal_link
- removed link qbhand2m1_ring_distal_virtual_link
- removed link qbhand2m1_ring_knuckle_link
- removed link qbhand2m1_ring_middle_link
- removed link qbhand2m1_ring_middle_virtual_link
- removed link qbhand2m1_ring_proximal_link
- removed link qbhand2m1_ring_proximal_virtual_link
- removed link qbhand2m1_synergy_tendon_virtual_link
- removed link qbhand2m1_thumb_distal_link
- removed link qbhand2m1_thumb_distal_virtual_link
- removed link qbhand2m1_thumb_knuckle_link
- removed link qbhand2m1_thumb_proximal_link
- removed link qbhand2m1_thumb_proximal_virtual_link
- added link box_link, mass 0.1; collision box size=0.75 0.75 0.94; visual box size=0.75 0.75 0.94
- added link panda_link0_sc
- added link panda_link1_sc
- added link panda_link2_sc
- added link panda_link3_sc
- added link panda_link4_sc
- added link panda_link5_sc
- added link panda_link6_sc
- added link panda_link7_sc
- added link qbhand1m_90_deg_flange_base_link, mass 0.205; collision mesh filename=package://qb_hand_description/meshes/flange_deg_90.stl scale=0.001 0.001 0.001; visual mesh filename=package://qb_hand_description/meshes/flange_deg_90.stl scale=0.001 0.001 0.001
- added link qbhand1m_base_link, mass 0.45; collision mesh filename=package://qb_hand_description/meshes/flange_iso_04.stl scale=0.001 0.001 0.001; visual mesh filename=package://qb_hand_description/meshes/flange_iso_04.stl scale=0.001 0.001 0.001
- added link qbhand1m_index_distal_link, mass 0.009; collision mesh filename=package://qb_hand_description/meshes/ph_distal_collision.stl scale=0.001 0.001 0.001; visual mesh filename=package://qb_hand_description/meshes/ph_distal.stl scale=0.001 0.001 0.001
- added link qbhand1m_index_distal_virtual_link, mass 1e-4
- added link qbhand1m_index_knuckle_link, mass 0.0095; collision mesh filename=package://qb_hand_description/meshes/ph_knuckle_collision.s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 scale=0.001 0.001 0.001; visual mesh filename=package://qb_hand_description/meshes/ph_knuckle.stl scale=0.001 0.001 0.001
- added link qbhand1m_index_middle_link, mass 0.0063; collision mesh filename=package://qb_hand_description/meshes/ph_short_collision.stl scale=0.001 0.001 0.001; visual mesh filename=package://qb_hand_description/meshes/ph_short.stl scale=0.001 0.001 0.001
- added link qbhand1m_index_middle_virtual_link, mass 1e-4
- added link qbhand1m_index_proximal_link, mass 0.0082; collision mesh filename=package://qb_hand_description/meshes/ph_medium_collision.stl scale=0.001 0.001 0.001; visual mesh filename=package://qb_hand_description/meshes/ph_medium.stl scale=0.001 0.001 0.001
- added link qbhand1m_index_proximal_virtual_link, mass 1e-4
- added link qbhand1m_little_distal_link, mass 0.009; collision mesh filename=package://qb_hand_description/meshes/ph_distal_collision.stl scale=0.001 0.001 0.001; visual mesh filename=package://qb_hand_description/meshes/ph_distal.stl scale=0.001 0.001 0.001
- added link qbhand1m_little_distal_virtual_link, mass 1e-4
- added link qbhand1m_little_knuckle_link, mass 0.0095; collision mesh filename=package://qb_hand_description/meshes/ph_knuckle_collision.s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 scale=0.001 0.001 0.001; visual mesh filename=package://qb_hand_description/meshes/ph_knuckle.stl scale=0.001 0.001 0.001
- added link qbhand1m_little_middle_link, mass 0.0063; collision mesh filename=package://qb_hand_description/meshes/ph_short_collision.stl scale=0.001 0.001 0.001; visual mesh filename=package://qb_hand_description/meshes/ph_short.stl scale=0.001 0.001 0.001
- added link qbhand1m_little_middle_virtual_link, mass 1e-4
- added link qbhand1m_little_proximal_link, mass 0.0063; collision mesh filename=package://qb_hand_description/meshes/ph_short_collision.stl scale=0.001 0.001 0.001; visual mesh filename=package://qb_hand_description/meshes/ph_short.stl scale=0.001 0.001 0.001
- added link qbhand1m_little_proximal_virtual_link, mass 1e-4
- added link qbhand1m_middle_distal_link, mass 0.009; collision mesh filename=package://qb_hand_description/meshes/ph_distal_collision.stl scale=0.001 0.001 0.001; visual mesh filename=package://qb_hand_description/meshes/ph_distal.stl scale=0.001 0.001 0.001
- added link qbhand1m_middle_distal_virtual_link, mass 1e-4
- added link qbhand1m_middle_knuckle_link, mass 0.0095; collision mesh filename=package://qb_hand_description/meshes/ph_knuckle_collision.s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 scale=0.001 0.001 0.001; visual mesh filename=package://qb_hand_description/meshes/ph_knuckle.stl scale=0.001 0.001 0.001
- added link qbhand1m_middle_middle_link, mass 0.0063; collision mesh filename=package://qb_hand_description/meshes/ph_short_collision.stl scale=0.001 0.001 0.001; visual mesh filename=package://qb_hand_description/meshes/ph_short.stl scale=0.001 0.001 0.001
- added link qbhand1m_middle_middle_virtual_link, mass 1e-4
- added link qbhand1m_middle_proximal_link, mass 0.0082; collision mesh filename=package://qb_hand_description/meshes/ph_medium_collision.stl scale=0.001 0.001 0.001; visual mesh filename=package://qb_hand_description/meshes/ph_medium.stl scale=0.001 0.001 0.001
- added link qbhand1m_middle_proximal_virtual_link, mass 1e-4
- added link qbhand1m_palm_link, mass 0.45; collision mesh filename=package://qb_hand_description/meshes/palm_pinch_r.stl scale=0.001 0.001 0.001; visual mesh filename=package://qb_hand_description/meshes/palm_pinch_r.stl scale=0.001 0.001 0.001
- added link qbhand1m_ring_distal_link, mass 0.009; collision mesh filename=package://qb_hand_description/meshes/ph_distal_collision.stl scale=0.001 0.001 0.001; visual mesh filename=package://qb_hand_description/meshes/ph_distal.stl scale=0.001 0.001 0.001
- added link qbhand1m_ring_distal_virtual_link, mass 1e-4
- added link qbhand1m_ring_knuckle_link, mass 0.0095; collision mesh filename=package://qb_hand_description/meshes/ph_knuckle_collision.s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 scale=0.001 0.001 0.001; visual mesh filename=package://qb_hand_description/meshes/ph_knuckle.stl scale=0.001 0.001 0.001
- added link qbhand1m_ring_middle_link, mass 0.0063; collision mesh filename=package://qb_hand_description/meshes/ph_short_collision.stl scale=0.001 0.001 0.001; visual mesh filename=package://qb_hand_description/meshes/ph_short.stl scale=0.001 0.001 0.001
- added link qbhand1m_ring_middle_virtual_link, mass 1e-4
- added link qbhand1m_ring_proximal_link, mass 0.0082; collision mesh filename=package://qb_hand_description/meshes/ph_medium_collision.stl scale=0.001 0.001 0.001; visual mesh filename=package://qb_hand_description/meshes/ph_medium.stl scale=0.001 0.001 0.001
- added link qbhand1m_ring_proximal_virtual_link, mass 1e-4
- added link qbhand1m_synergy_tendon_virtual_link, mass 1e-4
- added link qbhand1m_thumb_distal_link, mass 0.009; collision mesh filename=package://qb_hand_description/meshes/ph_distal_collision.stl scale=0.001 0.001 0.001; visual mesh filename=package://qb_hand_description/meshes/ph_distal.stl scale=0.001 0.001 0.001
- added link qbhand1m_thumb_distal_virtual_link, mass 1e-4
- added link qbhand1m_thumb_knuckle_link, mass 0.01; collision mesh filename=package://qb_hand_description/meshes/ph_thumb_r_collision.s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 scale=0.001 0.001 0.001; visual mesh filename=package://qb_hand_description/meshes/ph_thumb_r.stl scale=0.001 0.001 0.001
- added link qbhand1m_thumb_proximal_link, mass 0.0063; collision mesh filename=package://qb_hand_description/meshes/ph_short_collision.stl scale=0.001 0.001 0.001; visual mesh filename=package://qb_hand_description/meshes/ph_short.stl scale=0.001 0.001 0.001
- added link qbhand1m_thumb_proximal_virtual_link, mass 1e-4
- link panda_link0: mass 0.1 -> 0.629769; geometry collision mesh filename=package://franka_description/meshes/collision/link0.stl; visual mesh filename=package://franka_description/meshes/visual/link0.dae
- link panda_link1: mass 0.1 -> 4.970684; geometry collision mesh filename=package://franka_description/meshes/collision/link1.stl; visual mesh filename=package://franka_description/meshes/visual/link1.dae
- link panda_link2: mass 0.1 -> 0.646926; geometry collision mesh filename=package://franka_description/meshes/collision/link2.stl; visual mesh filename=package://franka_description/meshes/visual/link2.dae
- link panda_link3: mass 0.1 -> 3.228604; geometry collision mesh filename=package://franka_description/meshes/collision/link3.stl; visual mesh filename=package://franka_description/meshes/visual/link3.dae
- link panda_link4: mass 0.1 -> 3.587895; geometry collision mesh filename=package://franka_description/meshes/collision/link4.stl; visual mesh filename=package://franka_description/meshes/visual/link4.dae
- link panda_link5: mass 0.1 -> 1.225946; geometry collision mesh filename=package://franka_description/meshes/collision/link5.stl; visual mesh filename=package://franka_description/meshes/visual/link5.dae
- link panda_link6: mass 0.1 -> 1.666555; geometry collision mesh filename=package://franka_description/meshes/collision/link6.stl; visual mesh filename=package://franka_description/meshes/visual/link6.dae
- link panda_link7: mass 0.1 -> 0.735522; geometry collision mesh filename=package://franka_description/meshes/collision/link7.stl; visual mesh filename=package://franka_description/meshes/visual/link7.dae
- link panda_link8: mass 0.1 -> None; geometry 
Joints:
- removed joint qbhand2m1_90_deg_flange_base_fixed_joint
- removed joint qbhand2m1_base_fixed_joint
- removed joint qbhand2m1_index_distal_joint
- removed joint qbhand2m1_index_distal_virtual_joint
- removed joint qbhand2m1_index_knuckle_joint
- removed joint qbhand2m1_index_middle_joint
- removed joint qbhand2m1_index_middle_virtual_joint
- removed joint qbhand2m1_index_proximal_joint
- removed joint qbhand2m1_index_proximal_virtual_joint
- removed joint qbhand2m1_little_distal_joint
- removed joint qbhand2m1_little_distal_virtual_joint
- removed joint qbhand2m1_little_knuckle_joint
- removed joint qbhand2m1_little_middle_joint
- removed joint qbhand2m1_little_middle_virtual_joint
- removed joint qbhand2m1_little_proximal_joint
- removed joint qbhand2m1_little_proximal_virtual_joint
- removed joint qbhand2m1_manipulation_joint
- removed joint qbhand2m1_middle_distal_joint
- removed joint qbhand2m1_middle_distal_virtual_joint
- removed joint qbhand2m1_middle_knuckle_joint
- removed joint qbhand2m1_middle_middle_joint
- removed joint qbhand2m1_middle_middle_virtual_joint
- removed joint qbhand2m1_middle_proximal_joint
- removed joint qbhand2m1_middle_proximal_virtual_joint
- removed joint qbhand2m1_motor_1_joint
- removed joint qbhand2m1_motor_2_joint
- removed joint qbhand2m1_palm_fixed_joint
- removed joint qbhand2m1_ring_distal_joint
- removed joint qbhand2m1_ring_distal_virtual_joint
- removed joint qbhand2m1_ring_knuckle_joint
- removed joint qbhand2m1_ring_middle_joint
- removed joint qbhand2m1_ring_middle_virtual_joint
- removed joint qbhand2m1_ring_proximal_joint
- removed joint qbhand2m1_ring_proximal_virtual_joint
- removed joint qbhand2m1_synergy_joint
- removed joint qbhand2m1_thumb_distal_joint
- removed joint qbhand2m1_thumb_distal_virtual_joint
- removed joint qbhand2m1_thumb_knuckle_joint
- removed joint qbhand2m1_thumb_proximal_joint
- removed joint qbhand2m1_thumb_proximal_virtual_joint
- removed joint world_to_panda_joint
- added joint panda_joint: type fixed, parent box_link, child panda_link0, origin xyz=-0.18 0.0 0.47 rpy=0.0 0.0 0.0
- added joint panda_link0_sc_joint: type fixed, parent panda_link0, child panda_link0_sc, origin rpy=0 0 0
- added joint panda_link1_sc_joint: type fixed, parent panda_link1, child panda_link1_sc, origin rpy=0 0 0
- added joint panda_link2_sc_joint: type fixed, parent panda_link2, child panda_link2_sc, origin rpy=0 0 0
- added joint panda_link3_sc_joint: type fixed, parent panda_link3, child panda_link3_sc, origin rpy=0 0 0
- added joint panda_link4_sc_joint: type fixed, parent panda_link4, child panda_link4_sc, origin rpy=0 0 0
- added joint panda_link5_sc_joint: type fixed, parent panda_link5, child panda_link5_sc, origin rpy=0 0 0
- added joint panda_link6_sc_joint: type fixed, parent panda_link6, child panda_link6_sc, origin rpy=0 0 0
- added joint panda_link7_sc_joint: type fixed, parent panda_link7, child panda_link7_sc, origin rpy=0 0 0.7853981633974483
- added joint qbhand1m_90_deg_flange_base_fixed_joint: type fixed, parent qbhand1m_base_link, child qbhand1m_90_deg_flange_base_link, origin xyz=0 0 0 rpy=-1.57 0 0
- added joint qbhand1m_base_fixed_joint: type fixed, parent panda_link8, child qbhand1m_base_link, origin xyz=0.045 0 0.035 rpy=1.57 0 1.57
- added joint qbhand1m_index_distal_joint: type revolute, parent qbhand1m_index_middle_link, child qbhand1m_index_distal_virtual_link, origin xyz=0.009 0 0 rpy=0 0 0, axis 0 0 -1, limit lower=0.0 upper=0.785 effort=100 velocity=100, mimic joint=qbhand1m_synergy_joint multiplier=0.785
- added joint qbhand1m_index_distal_virtual_joint: type revolute, parent qbhand1m_index_distal_virtual_link, child qbhand1m_index_distal_link, origin xyz=0.013 0 0 rpy=0 0 0, axis 0 0 -1, limit lower=0.0 upper=0.785 effort=100 velocity=100, mimic joint=qbhand1m_index_distal_joint multiplier=1.0
- added joint qbhand1m_index_knuckle_joint: type revolute, parent qbhand1m_palm_link, child qbhand1m_index_knuckle_link, origin xyz=-0.02 -0.007 0.014 rpy=0 0 1.57, axis 0 0 -1, limit lower=-0.524 upper=0.524 effort=100 velocity=100, mimic joint=qbhand1m_synergy_joint multiplier=-0.2
- added joint qbhand1m_index_middle_joint: type revolute, parent qbhand1m_index_proximal_link, child qbhand1m_index_middle_virtual_link, origin xyz=0.017 0 0 rpy=0 0 0, axis 0 0 -1, limit lower=0.0 upper=0.785 effort=100 velocity=100, mimic joint=qbhand1m_synergy_joint multiplier=0.785
- added joint qbhand1m_index_middle_virtual_joint: type revolute, parent qbhand1m_index_middle_virtual_link, child qbhand1m_index_middle_link, origin xyz=0.013 0 0 rpy=0 0 0, axis 0 0 -1, limit lower=0.0 upper=0.785 effort=100 velocity=100, mimic joint=qbhand1m_index_middle_joint multiplier=1.0
- added joint qbhand1m_index_proximal_joint: type revolute, parent qbhand1m_index_knuckle_link, child qbhand1m_index_proximal_virtual_link, origin xyz=0.009 0 0 rpy=1.57 0 0, axis 0 0 -1, limit lower=0.0 upper=0.785 effort=100 velocity=100, mimic joint=qbhand1m_synergy_joint multiplier=0.785
- added joint qbhand1m_index_proximal_virtual_joint: type revolute, parent qbhand1m_index_proximal_virtual_link, child qbhand1m_index_proximal_link, origin xyz=0.013 0 0 rpy=0 0 0, axis 0 0 -1, limit lower=0.0 upper=0.785 effort=100 velocity=100, mimic joint=qbhand1m_index_proximal_joint multiplier=1.0
- added joint qbhand1m_little_distal_joint: type revolute, parent qbhand1m_little_middle_link, child qbhand1m_little_distal_virtual_link, origin xyz=0.009 0 0 rpy=0 0 0, axis 0 0 -1, limit lower=0.0 upper=0.785 effort=100 velocity=100, mimic joint=qbhand1m_synergy_joint multiplier=0.785
- added joint qbhand1m_little_distal_virtual_joint: type revolute, parent qbhand1m_little_distal_virtual_link, child qbhand1m_little_distal_link, origin xyz=0.013 0 0 rpy=0 0 0, axis 0 0 -1, limit lower=0.0 upper=0.785 effort=100 velocity=100, mimic joint=qbhand1m_little_distal_joint multiplier=1.0
- added joint qbhand1m_little_knuckle_joint: type revolute, parent qbhand1m_palm_link, child qbhand1m_little_knuckle_link, origin xyz=0.04 -0.012 0.014 rpy=0 0 1.57, axis 0 0 -1, limit lower=-0.524 upper=0.524 effort=100 velocity=100, mimic joint=qbhand1m_synergy_joint multiplier=0.4
- added joint qbhand1m_little_middle_joint: type revolute, parent qbhand1m_little_proximal_link, child qbhand1m_little_middle_virtual_link, origin xyz=0.009 0 0 rpy=0 0 0, axis 0 0 -1, limit lower=0.0 upper=0.785 effort=100 velocity=100, mimic joint=qbhand1m_synergy_joint multiplier=0.785
- added joint qbhand1m_little_middle_virtual_joint: type revolute, parent qbhand1m_little_middle_virtual_link, child qbhand1m_little_middle_link, origin xyz=0.013 0 0 rpy=0 0 0, axis 0 0 -1, limit lower=0.0 upper=0.785 effort=100 velocity=100, mimic joint=qbhand1m_little_middle_joint multiplier=1.0
- added joint qbhand1m_little_proximal_joint: type revolute, parent qbhand1m_little_knuckle_link, child qbhand1m_little_proximal_virtual_link, origin xyz=0.009 0 0 rpy=1.57 0 0, axis 0 0 -1, limit lower=0.0 upper=0.785 effort=100 velocity=100, mimic joint=qbhand1m_synergy_joint multiplier=0.785
- added joint qbhand1m_little_proximal_virtual_joint: type revolute, parent qbhand1m_little_proximal_virtual_link, child qbhand1m_little_proximal_link, origin xyz=0.013 0 0 rpy=0 0 0, axis 0 0 -1, limit lower=0.0 upper=0.785 effort=100 velocity=100, mimic joint=qbhand1m_little_proximal_joint multiplier=1.0
- added joint qbhand1m_middle_distal_joint: type revolute, parent qbhand1m_middle_middle_link, child qbhand1m_middle_distal_virtual_link, origin xyz=0.009 0 0 rpy=0 0 0, axis 0 0 -1, limit lower=0.0 upper=0.785 effort=100 velocity=100, mimic joint=qbhand1m_synergy_joint multiplier=0.785
- added joint qbhand1m_middle_distal_virtual_joint: type revolute, parent qbhand1m_middle_distal_virtual_link, child qbhand1m_middle_distal_link, origin xyz=0.013 0 0 rpy=0 0 0, axis 0 0 -1, limit lower=0.0 upper=0.785 effort=100 velocity=100, mimic joint=qbhand1m_middle_distal_joint multiplier=1.0
- added joint qbhand1m_middle_knuckle_joint: type revolute, parent qbhand1m_palm_link, child qbhand1m_middle_knuckle_link, origin xyz=0 0 0.014 rpy=0 0 1.57, axis 0 0 -1, limit lower=-0.524 upper=0.524 effort=100 velocity=100, mimic joint=qbhand1m_synergy_joint multiplier=0.0
- added joint qbhand1m_middle_middle_joint: type revolute, parent qbhand1m_middle_proximal_link, child qbhand1m_middle_middle_virtual_link, origin xyz=0.017 0 0 rpy=0 0 0, axis 0 0 -1, limit lower=0.0 upper=0.785 effort=100 velocity=100, mimic joint=qbhand1m_synergy_joint multiplier=0.785
- added joint qbhand1m_middle_middle_virtual_joint: type revolute, parent qbhand1m_middle_middle_virtual_link, child qbhand1m_middle_middle_link, origin xyz=0.013 0 0 rpy=0 0 0, axis 0 0 -1, limit lower=0.0 upper=0.785 effort=100 velocity=100, mimic joint=qbhand1m_middle_middle_joint multiplier=1.0
- added joint qbhand1m_middle_proximal_joint: type revolute, parent qbhand1m_middle_knuckle_link, child qbhand1m_middle_proximal_virtual_link, origin xyz=0.009 0 0 rpy=1.57 0 0, axis 0 0 -1, limit lower=0.0 upper=0.785 effort=100 velocity=100, mimic joint=qbhand1m_synergy_joint multiplier=0.785
- added joint qbhand1m_middle_proximal_virtual_joint: type revolute, parent qbhand1m_middle_proximal_virtual_link, child qbhand1m_middle_proximal_link, origin xyz=0.013 0 0 rpy=0 0 0, axis 0 0 -1, limit lower=0.0 upper=0.785 effort=100 velocity=100, mimic joint=qbhand1m_middle_proximal_joint multiplier=1.0
- added joint qbhand1m_palm_fixed_joint: type fixed, parent qbhand1m_base_link, child qbhand1m_palm_link, origin xyz=-0.0045 0.0145 0.144 rpy=1.57 0 0
- added joint qbhand1m_ring_distal_joint: type revolute, parent qbhand1m_ring_middle_link, child qbhand1m_ring_distal_virtual_link, origin xyz=0.009 0 0 rpy=0 0 0, axis 0 0 -1, limit lower=0.0 upper=0.785 effort=100 velocity=100, mimic joint=qbhand1m_synergy_joint multiplier=0.785
- added joint qbhand1m_ring_distal_virtual_joint: type revolute, parent qbhand1m_ring_distal_virtual_link, child qbhand1m_ring_distal_link, origin xyz=0.013 0 0 rpy=0 0 0, axis 0 0 -1, limit lower=0.0 upper=0.785 effort=100 velocity=100, mimic joint=qbhand1m_ring_distal_joint multiplier=1.0
- added joint qbhand1m_ring_knuckle_joint: type revolute, parent qbhand1m_palm_link, child qbhand1m_ring_knuckle_link, origin xyz=0.02 -0.007 0.014 rpy=0 0 1.57, axis 0 0 -1, limit lower=-0.524 upper=0.524 effort=100 velocity=100, mimic joint=qbhand1m_synergy_joint multiplier=0.2
- added joint qbhand1m_ring_middle_joint: type revolute, parent qbhand1m_ring_proximal_link, child qbhand1m_ring_middle_virtual_link, origin xyz=0.017 0 0 rpy=0 0 0, axis 0 0 -1, limit lower=0.0 upper=0.785 effort=100 velocity=100, mimic joint=qbhand1m_synergy_joint multiplier=0.785
- added joint qbhand1m_ring_middle_virtual_joint: type revolute, parent qbhand1m_ring_middle_virtual_link, child qbhand1m_ring_middle_link, origin xyz=0.013 0 0 rpy=0 0 0, axis 0 0 -1, limit lower=0.0 upper=0.785 effort=100 velocity=100, mimic joint=qbhand1m_ring_middle_joint multiplier=1.0
- added joint qbhand1m_ring_proximal_joint: type revolute, parent qbhand1m_ring_knuckle_link, child qbhand1m_ring_proximal_virtual_link, origin xyz=0.009 0 0 rpy=1.57 0 0, axis 0 0 -1, limit lower=0.0 upper=0.785 effort=100 velocity=100, mimic joint=qbhand1m_synergy_joint multiplier=0.785
- added joint qbhand1m_ring_proximal_virtual_joint: type revolute, parent qbhand1m_ring_proximal_virtual_link, child qbhand1m_ring_proximal_link, origin xyz=0.013 0 0 rpy=0 0 0, axis 0 0 -1, limit lower=0.0 upper=0.785 effort=100 velocity=100, mimic joint=qbhand1m_ring_proximal_joint multiplier=1.0
- added joint qbhand1m_synergy_joint: type revolute, parent qbhand1m_palm_link, child qbhand1m_synergy_tendon_virtual_link, origin xyz=0 0 0 rpy=0 0 0, axis 0 0 1, limit lower=0.0 upper=1.0 effort=100 velocity=100
- added joint qbhand1m_thumb_distal_joint: type revolute, parent qbhand1m_thumb_proximal_link, child qbhand1m_thumb_distal_virtual_link, origin xyz=0.009 0 0 rpy=0 0 0, axis 0 0 -1, limit lower=0.0 upper=0.785 effort=100 velocity=100, mimic joint=qbhand1m_synergy_joint multiplier=0.785
- added joint qbhand1m_thumb_distal_virtual_joint: type revolute, parent qbhand1m_thumb_distal_virtual_link, child qbhand1m_thumb_distal_link, origin xyz=0.013 0 0 rpy=0 0 0, axis 0 0 -1, limit lower=0.0 upper=0.785 effort=100 velocity=100, mimic joint=qbhand1m_thumb_distal_joint multiplier=1.0
- added joint qbhand1m_thumb_knuckle_joint: type revolute, parent qbhand1m_palm_link, child qbhand1m_thumb_knuckle_link, origin xyz=-0.044 -0.0465 -0.002 rpy=-1.57 3.14 0.0, axis 0 0 -1, limit lower=0.0 upper=1.571 effort=100 velocity=100, mimic joint=qbhand1m_synergy_joint multiplier=2.542
- added joint qbhand1m_thumb_proximal_joint: type revolute, parent qbhand1m_thumb_knuckle_link, child qbhand1m_thumb_proximal_virtual_link, origin xyz=0.0255 -0.0038 -0.00012 rpy=-1.1415 0.0 0.0, axis 0 0 -1, limit lower=0.0 upper=0.785 effort=100 velocity=100, mimic joint=qbhand1m_synergy_joint multiplier=0.785
- added joint qbhand1m_thumb_proximal_virtual_joint: type revolute, parent qbhand1m_thumb_proximal_virtual_link, child qbhand1m_thumb_proximal_link, origin xyz=0.013 0 0 rpy=0 0 0, axis 0 0 -1, limit lower=0.0 upper=0.785 effort=100 velocity=100, mimic joint=qbhand1m_thumb_proximal_joint multiplier=1.0
- added joint world_to_box_joint: type fixed, parent world, child box_link, origin xyz=0.0 0.0 0.47 rpy=0.0 0.0 0.0
- joint panda_joint1: limit lower=-2.8973 upper=2.8973 effort=87 velocity=2.1750 -> lower=-2.8973 upper=2.8973 effort=87.0 velocity=2.175
- joint panda_joint2: limit lower=-1.7628 upper=1.7628 effort=87 velocity=2.1750 -> lower=-1.7628 upper=1.7628 effort=87.0 velocity=2.175
- joint panda_joint3: limit lower=-2.8973 upper=2.8973 effort=87 velocity=2.1750 -> lower=-2.8973 upper=2.8973 effort=87.0 velocity=2.175
- joint panda_joint4: limit lower=-3.0718 upper=-0.0698 effort=87 velocity=2.1750 -> lower=-3.0718 upper=-0.0698 effort=87.0 velocity=2.175
- joint panda_joint5: limit lower=-2.8973 upper=2.8973 effort=12 velocity=2.6100 -> lower=-2.8973 upper=2.8973 effort=12.0 velocity=2.61
- joint panda_joint6: limit lower=-0.0175 upper=3.7525 effort=12 velocity=2.6100 -> lower=-0.0175 upper=3.7525 effort=12.0 velocity=2.61
- joint panda_joint7: limit lower=-2.8973 upper=2.8973 effort=12 velocity=2.6100 -> lower=-2.8973 upper=2.8973 effort=12.0 velocity=2.61
- joint right_hand_ee_joint: origin xyz=0.116 -0.002 0.036 rpy=0 0 0 -> xyz=0.102 -0.003 0.037 rpy=0 0 0
