Commit message: Added throwing, grasping, replacing task services for Bright/Makr Faire Demo 2022

File: panda_softhand_description/robot/panda_softhand.urdf.xacro (robot description, xacro)
@@ -7,4 +7,6 @@
   <xacro:include filename="$(find franka_description)/robots/panda_arm.xacro"/>
   <xacro:include filename="$(find soft_hand_description)/model/soft_hand_soma_panda.urdf.xacro"/>
+  <!-- con flangia -->
+  <!-- <xacro:include filename="$(find soft_hand_description)/model/soft_hand_darko_panda.urdf.xacro"/> -->
   <!-- WORLD -->
   <link name="world"/>
@@ -20,5 +22,5 @@
     <origin xyz="0 0 0" rpy="0 0 3.1415"/>
   </xacro:soft_hand_soma_panda>
-  <!-- EXTRA ENDEFFECTOR -->
+  <!-- EXTRA ENDEFFECTOR-CON FLANGIA ANGOLATA -->
   <joint name="right_hand_ee_joint" type="fixed">
     <origin xyz="0.130 0.000 0.035" rpy="0 0 0"/>
@@ -26,4 +28,10 @@
     <child link="right_hand_ee_link" />
   </joint>
+  <!-- EXTRA ENDEFFECTOR-SENZA FLANGIA -->
+  <!-- <joint name="right_hand_ee_joint" type="fixed">
+    <origin xyz="0.000 0.000 0.110" rpy="-1.5714 1.5714 0"/>
+    <parent link="panda_link8" />
+    <child link="right_hand_ee_link" />
+  </joint> -->
   <link name="right_hand_ee_link">
   </link>

Commit message: Several modifications from scratch to adapt to new melodic-devel of franka_ros and in line with the melodic-devel of panda_moveit_config

File: panda_softhand_description/robot/panda_softhand.urdf.xacro (robot description, xacro)
@@ -3,7 +3,7 @@
   <!-- ARGS -->
   <xacro:arg name="arm_id" default="panda"/>
-  <xacro:arg name="robot_ns" default="panda_arm"/>
+  <xacro:arg name="robot_ns" default="panda"/>
   <!-- MODELS -->
-  <xacro:include filename="$(find franka_description)/robots/panda_arm.xacro"/>
+  <xacro:include filename="$(find franka_description)/robots/common/franka_robot.xacro"/>
   <xacro:include filename="$(find soft_hand_description)/model/soft_hand_soma_panda.urdf.xacro"/>
   <!-- WORLD -->
@@ -15,5 +15,7 @@
   </joint>
   <!-- PANDA ARM -->
-  <xacro:panda_arm />
+  <xacro:franka_robot arm_id="$(arg arm_id)"
+                      joint_limits="${xacro.load_yaml('$(find franka_description)/robots/panda/joint_limits.yaml')}">
+  </xacro:franka_robot>
   <!-- RIGHT SOFTHAND -->
   <xacro:soft_hand_soma_panda parent="panda_link8" name="right_hand" left="false" withAdaptiveTransmission="true" useMimicTag="true">

File: panda_softhand_moveit_config/config/hand.xacro (robot description, xacro)
@@ -1,23 +1,45 @@
-<?xml version="1.0" ?>
+<?xml version="1.0" encoding="UTF-8"?>
 <robot xmlns:xacro="http://www.ros.org/wiki/xacro" name="panda">
-  <xacro:macro name="hand">
-    <!--GROUPS: Representation of a set of joints and links. This can be useful for specifying DOF to plan for, defining arms, end effectors, etc-->
-    <!--LINKS: When a link is specified, the parent joint of that link (if it exists) is automatically included-->
-    <!--JOINTS: When a joint is specified, the child link of that joint (which will always exist) is automatically included-->
-    <!--CHAINS: When a chain is specified, all the links along the chain (including endpoints) are included in the group. Additionally, all the joints that are parents to included links are also included. This means that joints along the chain and the parent joint of the base link are included in the group-->
-    <!--SUBGROUPS: Groups can also be formed by referencing to already defined group names-->
-    <group name="hand">
-      <link name="panda_hand" />
-      <link name="panda_leftfinger" />
-      <link name="panda_rightfinger" />
-      <joint name="panda_finger_joint1" />
-      <passive_joint name="panda_finger_joint2" />
-    </group>
-    <!--GROUP STATES: Purpose: Define a named state for a particular group, in terms of joint values. This is useful to define states like 'folded arms'-->
-    <!--END EFFECTOR: Purpose: Represent information about an end effector.-->
-    <!--DISABLE COLLISIONS: By default it is assumed that any link of the robot could potentially come into collision with any other link in the robot. This tag disables collision checking between a specified pair of links. -->
-    <disable_collisions link1="panda_hand" link2="panda_leftfinger" reason="Adjacent" />
-    <disable_collisions link1="panda_hand" link2="panda_rightfinger" reason="Adjacent" />
-    <disable_collisions link1="panda_leftfinger" link2="panda_rightfinger" reason="Default" />
-  </xacro:macro>
+    <xacro:macro name="hand">
+        <!--GROUPS: Representation of a set of joints and links. This can be useful for specifying DOF to plan for, defining arms, end effectors, etc-->
+        <!--LINKS: When a link is specified, the parent joint of that link (if it exists) is automatically included-->
+        <!--JOINTS: When a joint is specified, the child link of that joint (which will always exist) is automatically included-->
+        <!--CHAINS: When a chain is specified, all the links along the chain (including endpoints) are included in the group. Additionally, all the joints that are parents to included links are also included. This means that joints along the chain and the parent joint of the base link are included in the group-->
+        <!--SUBGROUPS: Groups can also be formed by referencing to already defined group names-->
+        <group name="$(arg arm_id)_hand">
+            <link name="$(arg arm_id)_hand"/>
+            <link name="$(arg arm_id)_leftfinger"/>
+            <link name="$(arg arm_id)_rightfinger"/>
+        </group>
+        <!--GROUP STATES: Purpose: Define a named state for a particular group, in terms of joint values. This is useful to define states like 'folded arms'-->
+        <group_state name="open" group="$(arg arm_id)_hand">
+            <joint name="$(arg arm_id)_finger_joint1" value="0.035"/>
+            <joint name="$(arg arm_id)_finger_joint2" value="0.035"/>
+        </group_state>
+        <group_state name="close" group="$(arg arm_id)_hand">
+            <joint name="$(arg arm_id)_finger_joint1" value="0"/>
+            <joint name="$(arg arm_id)_finger_joint2" value="0"/>
+        </group_state>
+        <!--END EFFECTOR: Purpose: Represent information about an end effector.-->
+        <!--VIRTUAL JOINT: Purpose: this element defines a virtual joint between a robot link and an external frame of reference (considered fixed with respect to the robot)-->
+        <!--PASSIVE JOINT: Purpose: this element is used to mark joints that are not actuated-->
+        <!--DISABLE COLLISIONS: By default it is assumed that any link of the robot could potentially come into collision with any other link in the robot. This tag disables collision checking between a specified pair of links. -->
+        <!-- Disable collision of hand link with all arm links. These are handled by the *_sc links -->
+        <xacro:property name="link_fmt" value="$(arg arm_id)_link{}" />
+        <xacro:disable_collisions_for link="$(arg arm_id)_hand" others="${[link_fmt.format(i) for i in python.range(8)]}" />
+        <xacro:disable_collisions_for link="$(arg arm_id)_hand_sc" others="${[link_fmt.format(i) for i in python.range(8)]}" />
+        <disable_collisions link1="$(arg arm_id)_hand_sc" link2="$(arg arm_id)_hand" reason="Never" />
+        <!-- Disable collision of fingers with all arm links -->
+        <xacro:property name="others" value="${[link_fmt.format(i) for i in python.range(8)] + [xacro.arg('arm_id') + '_hand', xacro.arg('arm_id') + '_hand_sc']}" />
+        <xacro:disable_collisions_for link="$(arg arm_id)_leftfinger" others="${list(others)}" />
+        <xacro:disable_collisions_for link="$(arg arm_id)_rightfinger" others="${list(others)}" />
+        <disable_collisions link1="$(arg arm_id)_leftfinger" link2="$(arg arm_id)_rightfinger" reason="Never" />
+        <!-- Disable collision of hand+fingers with all arm sc links -->
+        <xacro:property name="link_fmt" value="$(arg arm_id)_link{}_sc" />
+        <xacro:disable_collisions_for link="$(arg arm_id)_hand" others="${[link_fmt.format(i) for i in python.range(8)]}" />
+        <xacro:disable_collisions_for link="$(arg arm_id)_leftfinger" others="${[link_fmt.format(i) for i in python.range(8)]}" />
+        <xacro:disable_collisions_for link="$(arg arm_id)_rightfinger" others="${[link_fmt.format(i) for i in python.range(8)]}" />
+        <!-- Disable collision of hand_sc with selected arm sc links -->
+        <xacro:disable_collisions_for link="$(arg arm_id)_hand_sc" others="${[link_fmt.format(i) for i in [4,5,6,7]]}" />
+    </xacro:macro>
 </robot>
