Commit message: Several modifications from scratch to adapt to new melodic-devel of franka_ros and in line with the melodic-devel of panda_moveit_config

File: panda_softhand_moveit_config/config/panda.srdf.xacro (robot description, xacro)
@@ -1,50 +1,24 @@
-<?xml version="1.0" ?>
-<robot xmlns:xacro="http://www.ros.org/wiki/xacro" name="panda">
-  <xacro:macro name="panda_arm">
-    <!--GROUPS: Representation of a set of joints and links. This can be useful for specifying DOF to plan for, defining arms, end effectors, etc-->
-    <!--LINKS: When a link is specified, the parent joint of that link (if it exists) is automatically included-->
-    <!--JOINTS: When a joint is specified, the child link of that joint (which will always exist) is automatically included-->
-    <!--CHAINS: When a chain is specified, all the links along the chain (including endpoints) are included in the group. Additionally, all the joints that are parents to included links are also included. This means that joints along the chain and the parent joint of the base link are included in the group-->
-    <!--SUBGROUPS: Groups can also be formed by referencing to already defined group names-->
-    <group name="panda_arm">
-      <!-- <chain base_link="panda_link0" tip_link="panda_link8" /> -->
-      <chain base_link="panda_link0" tip_link="right_hand_ee_link" />
-    </group>
-    <!--GROUP STATES: Purpose: Define a named state for a particular group, in terms of joint values. This is useful to define states like 'folded arms'-->
-    <group_state name="ready" group="panda_arm">
-      <joint name="panda_joint1" value="0" />
-      <joint name="panda_joint2" value="-0.785" />
-      <joint name="panda_joint3" value="0" />
-      <joint name="panda_joint4" value="-2.356" />
-      <joint name="panda_joint5" value="0" />
-      <joint name="panda_joint6" value="1.571" />
-      <joint name="panda_joint7" value="0.785" />
-    </group_state>
-    <!--END EFFECTOR: Purpose: Represent information about an end effector.-->
-    <!--VIRTUAL JOINT: Purpose: this element defines a virtual joint between a robot link and an external frame of reference (considered fixed with respect to the robot)-->
-    <virtual_joint name="virtual_joint" type="floating" parent_frame="world" child_link="panda_link0" />
-    <!--DISABLE COLLISIONS: By default it is assumed that any link of the robot could potentially come into collision with any other link in the robot. This tag disables collision checking between a specified pair of links. -->
-    <disable_collisions link1="panda_link0" link2="panda_link1" reason="Adjacent" />
-    <disable_collisions link1="panda_link0" link2="panda_link2" reason="Never" />
-    <disable_collisions link1="panda_link0" link2="panda_link3" reason="Never" />
-    <disable_collisions link1="panda_link0" link2="panda_link4" reason="Never" />
-    <disable_collisions link1="panda_link1" link2="panda_link2" reason="Adjacent" />
-    <disable_collisions link1="panda_link1" link2="panda_link3" reason="Never" />
-    <disable_collisions link1="panda_link1" link2="panda_link4" reason="Never" />
-    <disable_collisions link1="panda_link2" link2="panda_link3" reason="Adjacent" />
-    <disable_collisions link1="panda_link2" link2="panda_link4" reason="Never" />
-    <disable_collisions link1="panda_link2" link2="panda_link6" reason="Never" />
-    <disable_collisions link1="panda_link3" link2="panda_link4" reason="Adjacent" />
-    <disable_collisions link1="panda_link3" link2="panda_link5" reason="Never" />
-    <disable_collisions link1="panda_link3" link2="panda_link6" reason="Never" />
-    <disable_collisions link1="panda_link3" link2="panda_link7" reason="Never" />
-    <disable_collisions link1="panda_link4" link2="panda_link5" reason="Adjacent" />
-    <disable_collisions link1="panda_link4" link2="panda_link6" reason="Never" />
-    <disable_collisions link1="panda_link4" link2="panda_link7" reason="Never" />
-    <disable_collisions link1="panda_link4" link2="panda_link8" reason="Never" />
-    <disable_collisions link1="panda_link5" link2="panda_link6" reason="Adjacent" />
-    <disable_collisions link1="panda_link6" link2="panda_link7" reason="Adjacent" />
-    <disable_collisions link1="panda_link6" link2="panda_link8" reason="Default" />
-    <disable_collisions link1="panda_link7" link2="panda_link8" reason="Adjacent" />
+<?xml version="1.0" encoding="UTF-8"?>
+<!--This does not replace URDF, and is not an extension of URDF.
+    This is a format for representing semantic information about the robot structure.
+    A URDF file must exist for this robot as well, where the joints and the links that are referenced are defined
+-->
+<robot xmlns:xacro="http://www.ros.org/wiki/xacro" name="panda_softhand">
+    <xacro:arg name="arm_id" default="panda" />
+    <xacro:include filename="$(find panda_softhand_moveit_config)/config/arm.xacro" />
+    <!-- panda_arm group: eef frame aligned to robot's flanche -->
+    <xacro:arm name="$(arg arm_id)_arm" tip_link="$(arg arm_id)_link8"/>
+    <!--Add the hand if people request it-->
+    <xacro:arg name="hand" default="false" />
+    <xacro:if value="$(arg hand)">
+        <!-- manipulator group: eef frame aligned to hand -->
+        <xacro:arm name="$(arg arm_id)_manipulator" tip_link="$(arg arm_id)_hand_tcp" />
+        <xacro:include filename="$(find panda_softhand_moveit_config)/config/hand.xacro" />
+        <xacro:hand />
+        <!--END EFFECTOR: Purpose: Represent information about an end effector.-->
+        <end_effector name="$(arg arm_id)_hand_tcp" parent_link="$(arg arm_id)_hand_tcp" group="$(arg arm_id)_hand" parent_group="$(arg arm_id)_manipulator" />
+        <!-- old end-effector -->
+        <end_effector name="$(arg arm_id)_hand" parent_link="$(arg arm_id)_link8" group="$(arg arm_id)_hand" parent_group="$(arg arm_id)_arm" />
+    </xacro:if>
     <!--ADDITIONALLY ADDED-->
     <passive_joint name="right_hand_index_abd_joint" />
@@ -236,4 +210,136 @@
     <disable_collisions link1="panda_link8" link2="right_hand_softhand_round_base" reason="Never" />
     <disable_collisions link1="panda_link8" link2="right_hand_panda_flange" reason="Never" />
+    <disable_collisions link1="panda_link2_sc" link2="right_hand_index_distal_link" reason="Never" />
+    <disable_collisions link1="panda_link2_sc" link2="right_hand_index_knuckle_link" reason="Never" />
+    <disable_collisions link1="panda_link2_sc" link2="right_hand_index_middle_link" reason="Never" />
+    <disable_collisions link1="panda_link2_sc" link2="right_hand_index_proximal_link" reason="Never" />
+    <disable_collisions link1="panda_link2_sc" link2="right_hand_little_distal_link" reason="Never" />
+    <disable_collisions link1="panda_link2_sc" link2="right_hand_little_knuckle_link" reason="Never" />
+    <disable_collisions link1="panda_link2_sc" link2="right_hand_little_middle_link" reason="Never" />
+    <disable_collisions link1="panda_link2_sc" link2="right_hand_little_proximal_link" reason="Never" />
+    <disable_collisions link1="panda_link2_sc" link2="right_hand_middle_distal_link" reason="Never" />
+    <disable_collisions link1="panda_link2_sc" link2="right_hand_middle_knuckle_link" reason="Never" />
+    <disable_collisions link1="panda_link2_sc" link2="right_hand_middle_middle_link" reason="Never" />
+    <disable_collisions link1="panda_link2_sc" link2="right_hand_middle_proximal_link" reason="Never" />
+    <disable_collisions link1="panda_link2_sc" link2="right_hand_palm_link" reason="Never" />
+    <disable_collisions link1="panda_link2_sc" link2="right_hand_ring_distal_link" reason="Never" />
+    <disable_collisions link1="panda_link2_sc" link2="right_hand_ring_knuckle_link" reason="Never" />
+    <disable_collisions link1="panda_link2_sc" link2="right_hand_ring_middle_link" reason="Never" />
+    <disable_collisions link1="panda_link2_sc" link2="right_hand_ring_proximal_link" reason="Never" />
+    <disable_collisions link1="panda_link2_sc" link2="right_hand_thumb_distal_link" reason="Never" />
+    <disable_collisions link1="panda_link2_sc" link2="right_hand_thumb_knuckle_link" reason="Never" />
+    <disable_collisions link1="panda_link2_sc" link2="right_hand_thumb_proximal_link" reason="Never" />
+    <disable_collisions link1="panda_link2_sc" link2="right_hand_softhand_round_base" reason="Never" />
+    <disable_collisions link1="panda_link2_sc" link2="right_hand_panda_flange" reason="Never" />
+    <disable_collisions link1="panda_link3_sc" link2="right_hand_index_distal_link" reason="Never" />
+    <disable_collisions link1="panda_link3_sc" link2="right_hand_index_knuckle_link" reason="Never" />
+    <disable_collisions link1="panda_link3_sc" link2="right_hand_index_middle_link" reason="Never" />
+    <disable_collisions link1="panda_link3_sc" link2="right_hand_index_proximal_link" reason="Never" />
+    <disable_collisions link1="panda_link3_sc" link2="right_hand_little_distal_link" reason="Never" />
+    <disable_collisions link1="panda_link3_sc" link2="right_hand_little_knuckle_link" reason="Never" />
+    <disable_collisions link1="panda_link3_sc" link2="right_hand_little_middle_link" reason="Never" />
+    <disable_collisions link1="panda_link3_sc" link2="right_hand_little_proximal_link" reason="Never" />
+    <disable_collisions link1="panda_link3_sc" link2="right_hand_middle_distal_link" reason="Never" />
+    <disable_collisions link1="panda_link3_sc" link2="right_hand_middle_knuckle_link" reason="Never" />
+    <disable_collisions link1="panda_link3_sc" link2="right_hand_middle_middle_link" reason="Never" />
+    <disable_collisions link1="panda_link3_sc" link2="right_hand_middle_proximal_link" reason="Never" />
+    <disable_collisions link1="panda_link3_sc" link2="right_hand_palm_link" reason="Never" />
+    <disable_collisions link1="panda_link3_sc" link2="right_hand_ring_distal_link" reason="Never" />
+    <disable_collisions link1="panda_link3_sc" link2="right_hand_ring_knuckle_link" reason="Never" />
+    <disable_collisions link1="panda_link3_sc" link2="right_hand_ring_middle_link" reason="Never" />
+    <disable_collisions link1="panda_link3_sc" link2="right_hand_ring_proximal_link" reason="Never" />
+    <disable_collisions link1="panda_link3_sc" link2="right_hand_thumb_distal_link" reason="Never" />
+    <disable_collisions link1="panda_link3_sc" link2="right_hand_thumb_knuckle_link" reason="Never" />
+    <disable_collisions link1="panda_link3_sc" link2="right_hand_thumb_proximal_link" reason="Never" />
+    <disable_collisions link1="panda_link3_sc" link2="right_hand_softhand_round_base" reason="Never" />
+    <disable_collisions link1="panda_link3_sc" link2="right_hand_panda_flange" reason="Never" />
+    <disable_collisions link1="panda_link4_sc" link2="right_hand_index_distal_link" reason="Never" />
+    <disable_collisions link1="panda_link4_sc" link2="right_hand_index_knuckle_link" reason="Never" />
+    <disable_collisions link1="panda_link4_sc" link2="right_hand_index_middle_link" reason="Never" />
+    <disable_collisions link1="panda_link4_sc" link2="right_hand_index_proximal_link" reason="Never" />
+    <disable_collisions link1="panda_link4_sc" link2="right_hand_little_distal_link" reason="Never" />
+    <disable_collisions link1="panda_link4_sc" link2="right_hand_little_knuckle_link" reason="Never" />
+    <disable_collisions link1="panda_link4_sc" link2="right_hand_little_middle_link" reason="Never" />
+    <disable_collisions link1="panda_link4_sc" link2="right_hand_little_proximal_link" reason="Never" />
+    <disable_collisions link1="panda_link4_sc" link2="right_hand_middle_distal_link" reason="Never" />
+    <disable_collisions link1="panda_link4_sc" link2="right_hand_middle_knuckle_link" reason="Never" />
+    <disable_collisions link1="panda_link4_sc" link2="right_hand_middle_middle_link" reason="Never" />
+    <disable_collisions link1="panda_link4_sc" link2="right_hand_middle_proximal_link" reason="Never" />
+    <disable_collisions link1="panda_link4_sc" link2="right_hand_palm_link" reason="Never" />
+    <disable_collisions link1="panda_link4_sc" link2="right_hand_ring_distal_link" reason="Never" />
+    <disable_collisions link1="panda_link4_sc" link2="right_hand_ring_knuckle_link" reason="Never" />
+    <disable_collisions link1="panda_link4_sc" link2="right_hand_ring_middle_link" reason="Never" />
+    <disable_collisions link1="panda_link4_sc" link2="right_hand_ring_proximal_link" reason="Never" />
+    <disable_collisions link1="panda_link4_sc" link2="right_hand_thumb_distal_link" reason="Never" />
+    <disable_collisions link1="panda_link4_sc" link2="right_hand_thumb_knuckle_link" reason="Never" />
+    <disable_collisions link1="panda_link4_sc" link2="right_hand_thumb_proximal_link" reason="Never" />
+    <disable_collisions link1="panda_link4_sc" link2="right_hand_softhand_round_base" reason="Never" />
+    <disable_collisions link1="panda_link4_sc" link2="right_hand_panda_flange" reason="Never" />
+    <disable_collisions link1="panda_link5_sc" link2="right_hand_index_distal_link" reason="Never" />
+    <disable_collisions link1="panda_link5_sc" link2="right_hand_index_knuckle_link" reason="Never" />
+    <disable_collisions link1="panda_link5_sc" link2="right_hand_index_middle_link" reason="Never" />
+    <disable_collisions link1="panda_link5_sc" link2="right_hand_index_proximal_link" reason="Never" />
+    <disable_collisions link1="panda_link5_sc" link2="right_hand_little_distal_link" reason="Never" />
+    <disable_collisions link1="panda_link5_sc" link2="right_hand_little_knuckle_link" reason="Never" />
+    <disable_collisions link1="panda_link5_sc" link2="right_hand_little_middle_link" reason="Never" />
+    <disable_collisions link1="panda_link5_sc" link2="right_hand_little_proximal_link" reason="Never" />
+    <disable_collisions link1="panda_link5_sc" link2="right_hand_middle_distal_link" reason="Never" />
+    <disable_collisions link1="panda_link5_sc" link2="right_hand_middle_knuckle_link" reason="Never" />
+    <disable_collisions link1="panda_link5_sc" link2="right_hand_middle_middle_link" reason="Never" />
+    <disable_collisions link1="panda_link5_sc" link2="right_hand_middle_proximal_link" reason="Never" />
+    <disable_collisions link1="panda_link5_sc" link2="right_hand_palm_link" reason="Never" />
+    <disable_collisions link1="panda_link5_sc" link2="right_hand_ring_distal_link" reason="Never" />
+    <disable_collisions link1="panda_link5_sc" link2="right_hand_ring_knuckle_link" reason="Never" />
+    <disable_collisions link1="panda_link5_sc" link2="right_hand_ring_middle_link" reason="Never" />
+    <disable_collisions link1="panda_link5_sc" link2="right_hand_ring_proximal_link" reason="Never" />
+    <disable_collisions link1="panda_link5_sc" link2="right_hand_thumb_distal_link" reason="Never" />
+    <disable_collisions link1="panda_link5_sc" link2="right_hand_thumb_knuckle_link" reason="Never" />
+    <disable_collisions link1="panda_link5_sc" link2="right_hand_thumb_proximal_link" reason="Never" />
+    <disable_collisions link1="panda_link5_sc" link2="right_hand_softhand_round_base" reason="Never" />
+    <disable_collisions link1="panda_link5_sc" link2="right_hand_panda_flange" reason="Never" />
+    <disable_collisions link1="panda_link6_sc" link2="right_hand_index_distal_link" reason="Never" />
+    <disable_collisions link1="panda_link6_sc" link2="right_hand_index_knuckle_link" reason="Never" />
+    <disable_collisions link1="panda_link6_sc" link2="right_hand_index_middle_link" reason="Never" />
+    <disable_collisions link1="panda_link6_sc" link2="right_hand_index_proximal_link" reason="Never" />
+    <disable_collisions link1="panda_link6_sc" link2="right_hand_little_distal_link" reason="Never" />
+    <disable_collisions link1="panda_link6_sc" link2="right_hand_little_knuckle_link" reason="Never" />
+    <disable_collisions link1="panda_link6_sc" link2="right_hand_little_middle_link" reason="Never" />
+    <disable_collisions link1="panda_link6_sc" link2="right_hand_little_proximal_link" reason="Never" />
+    <disable_collisions link1="panda_link6_sc" link2="right_hand_middle_distal_link" reason="Never" />
+    <disable_collisions link1="panda_link6_sc" link2="right_hand_middle_knuckle_link" reason="Never" />
+    <disable_collisions link1="panda_link6_sc" link2="right_hand_middle_middle_link" reason="Never" />
+    <disable_collisions link1="panda_link6_sc" link2="right_hand_middle_proximal_link" reason="Never" />
+    <disable_collisions link1="panda_link6_sc" link2="right_hand_palm_link" reason="Never" />
+    <disable_collisions link1="panda_link6_sc" link2="right_hand_ring_distal_link" reason="Never" />
+    <disable_collisions link1="panda_link6_sc" link2="right_hand_ring_knuckle_link" reason="Never" />
+    <disable_collisions link1="panda_link6_sc" link2="right_hand_ring_middle_link" reason="Never" />
+    <disable_collisions link1="panda_link6_sc" link2="right_hand_ring_proximal_link" reason="Never" />
+    <disable_collisions link1="panda_link6_sc" link2="right_hand_thumb_distal_link" reason="Never" />
+    <disable_collisions link1="panda_link6_sc" link2="right_hand_thumb_knuckle_link" reason="Never" />
+    <disable_collisions link1="panda_link6_sc" link2="right_hand_thumb_proximal_link" reason="Never" />
+    <disable_collisions link1="panda_link6_sc" link2="right_hand_softhand_round_base" reason="Never" />
+    <disable_collisions link1="panda_link6_sc" link2="right_hand_panda_flange" reason="Never" />
+    <disable_collisions link1="panda_link7_sc" link2="right_hand_index_distal_link" reason="Never" />
+    <disable_collisions link1="panda_link7_sc" link2="right_hand_index_knuckle_link" reason="Never" />
+    <disable_collisions link1="panda_link7_sc" link2="right_hand_index_middle_link" reason="Never" />
+    <disable_collisions link1="panda_link7_sc" link2="right_hand_index_proximal_link" reason="Never" />
+    <disable_collisions link1="panda_link7_sc" link2="right_hand_little_distal_link" reason="Never" />
+    <disable_collisions link1="panda_link7_sc" link2="right_hand_little_knuckle_link" reason="Never" />
+    <disable_collisions link1="panda_link7_sc" link2="right_hand_little_middle_link" reason="Never" />
+    <disable_collisions link1="panda_link7_sc" link2="right_hand_little_proximal_link" reason="Never" />
+    <disable_collisions link1="panda_link7_sc" link2="right_hand_middle_distal_link" reason="Never" />
+    <disable_collisions link1="panda_link7_sc" link2="right_hand_middle_knuckle_link" reason="Never" />
+    <disable_collisions link1="panda_link7_sc" link2="right_hand_middle_middle_link" reason="Never" />
+    <disable_collisions link1="panda_link7_sc" link2="right_hand_middle_proximal_link" reason="Never" />
+    <disable_collisions link1="panda_link7_sc" link2="right_hand_palm_link" reason="Never" />
+    <disable_collisions link1="panda_link7_sc" link2="right_hand_ring_distal_link" reason="Never" />
+    <disable_collisions link1="panda_link7_sc" link2="right_hand_ring_knuckle_link" reason="Never" />
+    <disable_collisions link1="panda_link7_sc" link2="right_hand_ring_middle_link" reason="Never" />
+    <disable_collisions link1="panda_link7_sc" link2="right_hand_ring_proximal_link" reason="Never" />
+    <disable_collisions link1="panda_link7_sc" link2="right_hand_thumb_distal_link" reason="Never" />
+    <disable_collisions link1="panda_link7_sc" link2="right_hand_thumb_knuckle_link" reason="Never" />
+    <disable_collisions link1="panda_link7_sc" link2="right_hand_thumb_proximal_link" reason="Never" />
+    <disable_collisions link1="panda_link7_sc" link2="right_hand_softhand_round_base" reason="Never" />
+    <disable_collisions link1="panda_link7_sc" link2="right_hand_panda_flange" reason="Never" />
     <disable_collisions link1="right_hand_panda_flange" link2="right_hand_index_distal_link" reason="Never" />
     <disable_collisions link1="right_hand_panda_flange" link2="right_hand_index_knuckle_link" reason="Never" />
@@ -468,4 +574,3 @@
     <disable_collisions link1="right_hand_thumb_distal_link" link2="right_hand_thumb_proximal_link" reason="Adjacent" />
     <disable_collisions link1="right_hand_thumb_knuckle_link" link2="right_hand_thumb_proximal_link" reason="Adjacent" />
-  </xacro:macro>
 </robot>

Commit message: Added panda_softhand_msgs for the definition of srvs. Created from scratch (SetupAssistant) the moveit_config pkg (with the hand taken from the xacro utils)

File: panda_softhand_description/robot/panda_softhand.urdf.xacro (robot description, xacro)
@@ -3,8 +3,8 @@
   <!-- ARGS -->
   <xacro:arg name="arm_id" default="panda"/>
-  <xacro:arg name="robot_ns" default="panda_arm"/>
+  <xacro:arg name="robot_ns" default="panda"/>
   <!-- MODELS -->
-  <xacro:include filename="$(find franka_description)/robots/panda_arm.xacro"/>
-  <xacro:include filename="$(find soft_hand_description)/model/soft_hand_soma_panda.urdf.xacro"/>
+  <xacro:include filename="$(find franka_description)/robots/common/franka_robot.xacro"/>
+  <xacro:include filename="$(find qb_hand_description)/urdf/qbhand.utils.xacro"/>
   <!-- WORLD -->
   <link name="world"/>
@@ -15,12 +15,15 @@
   </joint>
   <!-- PANDA ARM -->
-  <xacro:panda_arm />
+  <xacro:franka_robot arm_id="$(arg arm_id)"
+      joint_limits="${xacro.load_yaml('$(find franka_description)/robots/panda/joint_limits.yaml')}">
+  </xacro:franka_robot>
   <!-- RIGHT SOFTHAND -->
-  <xacro:soft_hand_soma_panda parent="panda_link8" name="right_hand" left="false" withAdaptiveTransmission="true" useMimicTag="true">
-    <origin xyz="0 0 0" rpy="0 0 3.1415"/>
-  </xacro:soft_hand_soma_panda>
+  <xacro:arg name="namespace" default="qbhand2m1"/>
+  <xacro:build_hand_2m_from_yaml_with_90_deg_flange configuration="qbhand_right" namespace="$(arg namespace)" parent="panda_link8" parent_link_suffix="">
+		  <origin xyz="0.045 0 0.035" rpy="1.57 0 1.57"/>
+	</xacro:build_hand_2m_from_yaml_with_90_deg_flange>
   <!-- EXTRA ENDEFFECTOR -->
   <joint name="right_hand_ee_joint" type="fixed">
-    <origin xyz="0.130 0.000 0.035" rpy="0 0 0"/>
+    <origin xyz="0.116 -0.002 0.036" rpy="0 0 0"/>
     <parent link="panda_link8" />
     <child link="right_hand_ee_link" />
