Commit message: Changed panda_softhand_moveit_config and the franka_ros pkg(taken from the zip on the Darko Platform)

File: panda_softhand_description/robot/panda_softhand.urdf.xacro (robot description, xacro)
@@ -5,5 +5,5 @@
   <xacro:arg name="robot_ns" default="panda"/>
   <!-- MODELS -->
-  <xacro:include filename="$(find franka_description)/robots/common/franka_robot.xacro"/>
+  <xacro:include filename="$(find franka_description)/robots/panda_arm.xacro"/>
   <xacro:include filename="$(find qb_hand_description)/urdf/qbhand.utils.xacro"/>
   <!-- WORLD -->
@@ -15,8 +15,6 @@
   </joint>
   <!-- PANDA ARM -->
-  <xacro:franka_robot arm_id="$(arg arm_id)"
-      joint_limits="${xacro.load_yaml('$(find franka_description)/robots/panda/joint_limits.yaml')}">
-  </xacro:franka_robot>
-  <!-- RIGHT SOFTHAND -->
+  <xacro:panda_arm/>
+  <!-- RIGHT SOFTHAND2 -->
   <xacro:arg name="namespace" default="qbhand2m1"/>
   <xacro:build_hand_2m_from_yaml_with_90_deg_flange configuration="qbhand_right" namespace="$(arg namespace)" parent="panda_link8" parent_link_suffix="">

File: panda_softhand_moveit_config/config/gazebo_panda_softhand.urdf (robot description, URDF)
Before this commit: robot panda_softhand, 59 links, 58 joints
Links:
- removed link panda_link0_sc
- removed link panda_link1_sc
- removed link panda_link2_sc
- removed link panda_link3_sc
- removed link panda_link4_sc
- removed link panda_link5_sc
- removed link panda_link6_sc
- removed link panda_link7_sc
- link panda_link0: geometry collision cylinder length=0.03 radius=0.06; collision sphere radius=0.06
- link panda_link1: geometry collision cylinder length=0.2830 radius=0.06; collision sphere radius=0.06
- link panda_link2: geometry collision cylinder length=0.12 radius=0.06; collision sphere radius=0.06
- link panda_link3: geometry collision cylinder length=0.15 radius=0.06; collision sphere radius=0.06
- link panda_link4: geometry collision cylinder length=0.12 radius=0.06; collision sphere radius=0.06
- link panda_link5: geometry collision cylinder length=0.1 radius=0.06; collision cylinder length=0.14 radius=0.025
- link panda_link6: geometry collision cylinder length=0.08 radius=0.05; collision sphere radius=0.05
- link panda_link7: geometry collision cylinder length=0.14 radius=0.04; collision sphere radius=0.04
- link panda_link8: mass None -> 0.1; geometry collision cylinder length=0.01 radius=0.03; collision sphere radius=0.03
Joints:
- removed joint panda_link0_sc_joint
- removed joint panda_link1_sc_joint
- removed joint panda_link2_sc_joint
- removed joint panda_link3_sc_joint
- removed joint panda_link4_sc_joint
- removed joint panda_link5_sc_joint
- removed joint panda_link6_sc_joint
- removed joint panda_link7_sc_joint
- joint panda_joint1: limit lower=-2.8973 upper=2.8973 effort=87.0 velocity=2.175 -> lower=-2.8973 upper=2.8973 effort=87 velocity=2.1750
- joint panda_joint2: limit lower=-1.7628 upper=1.7628 effort=87.0 velocity=2.175 -> lower=-1.7628 upper=1.7628 effort=87 velocity=2.1750
- joint panda_joint3: limit lower=-2.8973 upper=2.8973 effort=87.0 velocity=2.175 -> lower=-2.8973 upper=2.8973 effort=87 velocity=2.1750
- joint panda_joint4: limit lower=-3.0718 upper=-0.0698 effort=87.0 velocity=2.175 -> lower=-3.0718 upper=-0.0698 effort=87 velocity=2.1750
- joint panda_joint5: limit lower=-2.8973 upper=2.8973 effort=12.0 velocity=2.61 -> lower=-2.8973 upper=2.8973 effort=12 velocity=2.6100
- joint panda_joint6: limit lower=-0.0175 upper=3.7525 effort=12.0 velocity=2.61 -> lower=-0.0175 upper=3.7525 effort=12 velocity=2.6100
- joint panda_joint7: limit lower=-2.8973 upper=2.8973 effort=12.0 velocity=2.61 -> lower=-2.8973 upper=2.8973 effort=12 velocity=2.6100
