Commit message: Pick seems working

File: panda_softhand_description/robot/arm/darko_franka_robot.xacro (robot description, xacro)
@@ -4,5 +4,5 @@
     <!-- Name of this panda -->
     <!-- Should a franka_gripper be mounted at the flange?" -->
-    <xacro:arg name="hand" default="true" />
+    <xacro:arg name="hand" default="false" />
     <!-- Positional offset between $(arm_id)_hand -> $(arm_id)_hand_tcp [m]. Only used when
     hand:=true -->
@@ -12,5 +12,5 @@
     <xacro:arg name="tcp_rpy" default="0 0 0" />
     <!-- Is the robot being simulated in gazebo?" -->
-    <xacro:arg name="gazebo" default="true" />
+    <xacro:arg name="gazebo" default="false" />
     <xacro:include filename="$(find franka_description)/robots/common/utils.xacro" />
     <xacro:include filename="$(find franka_description)/robots/common/franka_arm.xacro" />

File: panda_softhand_description/robot/urdf/panda_softhand.urdf.xacro (robot description, xacro)
@@ -50,16 +50,21 @@
       rpy="${arm_orientation_r} ${arm_orientation_p} ${arm_orientation_y}" />
   </xacro:darko_franka_robot>
-  <!-- RIGHT SOFTHAND2 -->
-  <xacro:arg
-    name="namespace" default="qbhand1m" />
-  <xacro:build_hand_from_yaml_with_90_deg_flange
-    configuration="qbhand_right"
+  <!-- <joint
+    name="panda_link8_to_root_link_joint" type="fixed">
+    <origin xyz="0.0 0.0 0.0" rpy="0.0 0.0 0.0" />
+    <parent link="panda_link8" />
+    <child link="root_link" />
+  </joint>
+  <link name="root_link" /> -->
+  <!-- RIGHT SOFTHAND1 -->
+  <xacro:arg name="namespace" default="qbhand1" />
+  <xacro:build_hand_from_yaml_with_90_deg_flange configuration="qbhand_right"
     namespace="$(arg namespace)" parent="panda_link8" parent_link_suffix="">
     <origin xyz="0.045 0 0.035" rpy="1.57 0 1.57" />
   </xacro:build_hand_from_yaml_with_90_deg_flange>
-  <!-- EXTRA ENDEFFECTOR -->
+  <!-- EXTRA ENDEFFECTOR Classical one -->
   <joint
     name="right_hand_ee_joint" type="fixed">
-    <origin xyz="0.102 -0.003 0.037" rpy="0 0 0" />
+    <origin xyz="0.13 -0.003 0.037" rpy="0 0 0" />
     <parent link="panda_link8" />
     <child link="right_hand_ee_link" />
@@ -67,3 +72,10 @@
   <link name="right_hand_ee_link">
   </link>
+  <!-- Thumb index ee link frame -->
+  <link name="thumb_index_ee_link" />
+  <joint name="thumb_index_ee_joint" type="fixed">
+    <origin xyz="0.07 -0.04 0.03" rpy="0 0.5 -1.0" />
+    <parent link="right_hand_ee_link" />
+    <child link="thumb_index_ee_link" />
+  </joint>
 </robot>

File: panda_softhand_description/robot/utils/properties.xacro (robot description, xacro)
@@ -8,5 +8,5 @@
     <xacro:property name="base_height" value="0.94" />
     <!-- Define arm base position -->
-    <xacro:property name="arm_position_x" value="-0.18" />
+    <xacro:property name="arm_position_x" value="0.12" />
     <xacro:property name="arm_position_y" value="0.0" />
     <xacro:property name="arm_position_z" value="0.0" />
