Commit message: Pick seems working

File: panda_softhand_moveit_config/config/gazebo_panda_softhand.urdf (robot description, URDF)
Before this commit: robot panda_softhand, 57 links, 56 joints
Links:
- removed link qbhand1m_90_deg_flange_base_link
- removed link qbhand1m_base_link
- removed link qbhand1m_index_distal_link
- removed link qbhand1m_index_distal_virtual_link
- removed link qbhand1m_index_knuckle_link
- removed link qbhand1m_index_middle_link
- removed link qbhand1m_index_middle_virtual_link
- removed link qbhand1m_index_proximal_link
- removed link qbhand1m_index_proximal_virtual_link
- removed link qbhand1m_little_distal_link
- removed link qbhand1m_little_distal_virtual_link
- removed link qbhand1m_little_knuckle_link
- removed link qbhand1m_little_middle_link
- removed link qbhand1m_little_middle_virtual_link
- removed link qbhand1m_little_proximal_link
- removed link qbhand1m_little_proximal_virtual_link
- removed link qbhand1m_middle_distal_link
- removed link qbhand1m_middle_distal_virtual_link
- removed link qbhand1m_middle_knuckle_link
- removed link qbhand1m_middle_middle_link
- removed link qbhand1m_middle_middle_virtual_link
- removed link qbhand1m_middle_proximal_link
- removed link qbhand1m_middle_proximal_virtual_link
- removed link qbhand1m_palm_link
- removed link qbhand1m_ring_distal_link
- removed link qbhand1m_ring_distal_virtual_link
- removed link qbhand1m_ring_knuckle_link
- removed link qbhand1m_ring_middle_link
- removed link qbhand1m_ring_middle_virtual_link
- removed link qbhand1m_ring_proximal_link
- removed link qbhand1m_ring_proximal_virtual_link
- removed link qbhand1m_synergy_tendon_virtual_link
- removed link qbhand1m_thumb_distal_link
- removed link qbhand1m_thumb_distal_virtual_link
- removed link qbhand1m_thumb_knuckle_link
- removed link qbhand1m_thumb_proximal_link
- removed link qbhand1m_thumb_proximal_virtual_link
- added link qbhand1_90_deg_flange_base_link, mass 0.205; collision mesh filename=package://qb_hand_description/meshes/flange_deg_90.stl scale=0.001 0.001 0.001; visual mesh filename=package://qb_hand_description/meshes/flange_deg_90.stl scale=0.001 0.001 0.001
- added link qbhand1_base_link, mass 0.45; collision mesh filename=package://qb_hand_description/meshes/flange_iso_04.stl scale=0.001 0.001 0.001; visual mesh filename=package://qb_hand_description/meshes/flange_iso_04.stl scale=0.001 0.001 0.001
- added link qbhand1_index_distal_link, mass 0.009; collision mesh filename=package://qb_hand_description/meshes/ph_distal_collision.stl scale=0.001 0.001 0.001; visual mesh filename=package://qb_hand_description/meshes/ph_distal.stl scale=0.001 0.001 0.001
- added link qbhand1_index_distal_virtual_link, mass 1e-4
- added link qbhand1_index_knuckle_link, mass 0.0095; collision mesh filename=package://qb_hand_description/meshes/ph_knuckle_collision.s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 scale=0.001 0.001 0.001; visual mesh filename=package://qb_hand_description/meshes/ph_knuckle.stl scale=0.001 0.001 0.001
- added link qbhand1_index_middle_link, mass 0.0063; collision mesh filename=package://qb_hand_description/meshes/ph_short_collision.stl scale=0.001 0.001 0.001; visual mesh filename=package://qb_hand_description/meshes/ph_short.stl scale=0.001 0.001 0.001
- added link qbhand1_index_middle_virtual_link, mass 1e-4
- added link qbhand1_index_proximal_link, mass 0.0082; collision mesh filename=package://qb_hand_description/meshes/ph_medium_collision.stl scale=0.001 0.001 0.001; visual mesh filename=package://qb_hand_description/meshes/ph_medium.stl scale=0.001 0.001 0.001
- added link qbhand1_index_proximal_virtual_link, mass 1e-4
- added link qbhand1_little_distal_link, mass 0.009; collision mesh filename=package://qb_hand_description/meshes/ph_distal_collision.stl scale=0.001 0.001 0.001; visual mesh filename=package://qb_hand_description/meshes/ph_distal.stl scale=0.001 0.001 0.001
- added link qbhand1_little_distal_virtual_link, mass 1e-4
- added link qbhand1_little_knuckle_link, mass 0.0095; collision mesh filename=package://qb_hand_description/meshes/ph_knuckle_collision.s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 scale=0.001 0.001 0.001; visual mesh filename=package://qb_hand_description/meshes/ph_knuckle.stl scale=0.001 0.001 0.001
- added link qbhand1_little_middle_link, mass 0.0063; collision mesh filename=package://qb_hand_description/meshes/ph_short_collision.stl scale=0.001 0.001 0.001; visual mesh filename=package://qb_hand_description/meshes/ph_short.stl scale=0.001 0.001 0.001
- added link qbhand1_little_middle_virtual_link, mass 1e-4
- added link qbhand1_little_proximal_link, mass 0.0063; collision mesh filename=package://qb_hand_description/meshes/ph_short_collision.stl scale=0.001 0.001 0.001; visual mesh filename=package://qb_hand_description/meshes/ph_short.stl scale=0.001 0.001 0.001
- added link qbhand1_little_proximal_virtual_link, mass 1e-4
- added link qbhand1_middle_distal_link, mass 0.009; collision mesh filename=package://qb_hand_description/meshes/ph_distal_collision.stl scale=0.001 0.001 0.001; visual mesh filename=package://qb_hand_description/meshes/ph_distal.stl scale=0.001 0.001 0.001
- added link qbhand1_middle_distal_virtual_link, mass 1e-4
- added link qbhand1_middle_knuckle_link, mass 0.0095; collision mesh filename=package://qb_hand_description/meshes/ph_knuckle_collision.s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 scale=0.001 0.001 0.001; visual mesh filename=package://qb_hand_description/meshes/ph_knuckle.stl scale=0.001 0.001 0.001
- added link qbhand1_middle_middle_link, mass 0.0063; collision mesh filename=package://qb_hand_description/meshes/ph_short_collision.stl scale=0.001 0.001 0.001; visual mesh filename=package://qb_hand_description/meshes/ph_short.stl scale=0.001 0.001 0.001
- added link qbhand1_middle_middle_virtual_link, mass 1e-4
- added link qbhand1_middle_proximal_link, mass 0.0082; collision mesh filename=package://qb_hand_description/meshes/ph_medium_collision.stl scale=0.001 0.001 0.001; visual mesh filename=package://qb_hand_description/meshes/ph_medium.stl scale=0.001 0.001 0.001
- added link qbhand1_middle_proximal_virtual_link, mass 1e-4
- added link qbhand1_palm_link, mass 0.45; collision mesh filename=package://qb_hand_description/meshes/palm_pinch_r.stl scale=0.001 0.001 0.001; visual mesh filename=package://qb_hand_description/meshes/palm_pinch_r.stl scale=0.001 0.001 0.001
- added link qbhand1_ring_distal_link, mass 0.009; collision mesh filename=package://qb_hand_description/meshes/ph_distal_collision.stl scale=0.001 0.001 0.001; visual mesh filename=package://qb_hand_description/meshes/ph_distal.stl scale=0.001 0.001 0.001
- added link qbhand1_ring_distal_virtual_link, mass 1e-4
- added link qbhand1_ring_knuckle_link, mass 0.0095; collision mesh filename=package://qb_hand_description/meshes/ph_knuckle_collision.s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 scale=0.001 0.001 0.001; visual mesh filename=package://qb_hand_description/meshes/ph_knuckle.stl scale=0.001 0.001 0.001
- added link qbhand1_ring_middle_link, mass 0.0063; collision mesh filename=package://qb_hand_description/meshes/ph_short_collision.stl scale=0.001 0.001 0.001; visual mesh filename=package://qb_hand_description/meshes/ph_short.stl scale=0.001 0.001 0.001
- added link qbhand1_ring_middle_virtual_link, mass 1e-4
- added link qbhand1_ring_proximal_link, mass 0.0082; collision mesh filename=package://qb_hand_description/meshes/ph_medium_collision.stl scale=0.001 0.001 0.001; visual mesh filename=package://qb_hand_description/meshes/ph_medium.stl scale=0.001 0.001 0.001
- added link qbhand1_ring_proximal_virtual_link, mass 1e-4
- added link qbhand1_synergy_tendon_virtual_link, mass 1e-4
- added link qbhand1_thumb_distal_link, mass 0.009; collision mesh filename=package://qb_hand_description/meshes/ph_distal_collision.stl scale=0.001 0.001 0.001; visual mesh filename=package://qb_hand_description/meshes/ph_distal.stl scale=0.001 0.001 0.001
- added link qbhand1_thumb_distal_virtual_link, mass 1e-4
- added link qbhand1_thumb_knuckle_link, mass 0.01; collision mesh filename=package://qb_hand_description/meshes/ph_thumb_r_collision.s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 scale=0.001 0.001 0.001; visual mesh filename=package://qb_hand_description/meshes/ph_thumb_r.stl scale=0.001 0.001 0.001
- added link qbhand1_thumb_proximal_link, mass 0.0063; collision mesh filename=package://qb_hand_description/meshes/ph_short_collision.stl scale=0.001 0.001 0.001; visual mesh filename=package://qb_hand_description/meshes/ph_short.stl scale=0.001 0.001 0.001
- added link qbhand1_thumb_proximal_virtual_link, mass 1e-4
- added link thumb_index_ee_link
- link panda_link0: mass 0.629769 -> 0.1
- link panda_link0_sc: mass None -> 0.1; geometry collision cylinder length=0.03 radius=0.09; collision sphere radius=0.09
- link panda_link1: mass 4.970684 -> 0.1
- link panda_link1_sc: mass None -> 0.1; geometry collision cylinder length=0.283 radius=0.09; collision sphere radius=0.09
- link panda_link2: mass 0.646926 -> 0.1
- link panda_link2_sc: mass None -> 0.1; geometry collision cylinder length=0.12 radius=0.09; collision sphere radius=0.09
- link panda_link3: mass 3.228604 -> 0.1
- link panda_link3_sc: mass None -> 0.1; geometry collision cylinder length=0.15 radius=0.09; collision sphere radius=0.09
- link panda_link4: mass 3.587895 -> 0.1
- link panda_link4_sc: mass None -> 0.1; geometry collision cylinder length=0.12 radius=0.09; collision sphere radius=0.09
- link panda_link5: mass 1.225946 -> 0.1
- link panda_link5_sc: mass None -> 0.1; geometry collision cylinder length=0.1 radius=0.09; collision cylinder length=0.14 radius=0.055
- link panda_link6: mass 1.666555 -> 0.1
- link panda_link6_sc: mass None -> 0.1; geometry collision cylinder length=0.08 radius=0.08; collision sphere radius=0.08
- link panda_link7: mass 0.735522 -> 0.1
- link panda_link7_sc: mass None -> 0.1; geometry collision cylinder length=0.01 radius=0.06; collision cylinder length=0.14 radius=0.07
Joints:
- removed joint qbhand1m_90_deg_flange_base_fixed_joint
- removed joint qbhand1m_base_fixed_joint
- removed joint qbhand1m_index_distal_joint
- removed joint qbhand1m_index_distal_virtual_joint
- removed joint qbhand1m_index_knuckle_joint
- removed joint qbhand1m_index_middle_joint
- removed joint qbhand1m_index_middle_virtual_joint
- removed joint qbhand1m_index_proximal_joint
- removed joint qbhand1m_index_proximal_virtual_joint
- removed joint qbhand1m_little_distal_joint
- removed joint qbhand1m_little_distal_virtual_joint
- removed joint qbhand1m_little_knuckle_joint
- removed joint qbhand1m_little_middle_joint
- removed joint qbhand1m_little_middle_virtual_joint
- removed joint qbhand1m_little_proximal_joint
- removed joint qbhand1m_little_proximal_virtual_joint
- removed joint qbhand1m_middle_distal_joint
- removed joint qbhand1m_middle_distal_virtual_joint
- removed joint qbhand1m_middle_knuckle_joint
- removed joint qbhand1m_middle_middle_joint
- removed joint qbhand1m_middle_middle_virtual_joint
- removed joint qbhand1m_middle_proximal_joint
- removed joint qbhand1m_middle_proximal_virtual_joint
- removed joint qbhand1m_palm_fixed_joint
- removed joint qbhand1m_ring_distal_joint
- removed joint qbhand1m_ring_distal_virtual_joint
- removed joint qbhand1m_ring_knuckle_joint
- removed joint qbhand1m_ring_middle_joint
- removed joint qbhand1m_ring_middle_virtual_joint
- removed joint qbhand1m_ring_proximal_joint
- removed joint qbhand1m_ring_proximal_virtual_joint
- removed joint qbhand1m_synergy_joint
- removed joint qbhand1m_thumb_distal_joint
- removed joint qbhand1m_thumb_distal_virtual_joint
- removed joint qbhand1m_thumb_knuckle_joint
- removed joint qbhand1m_thumb_proximal_joint
- removed joint qbhand1m_thumb_proximal_virtual_joint
- added joint qbhand1_90_deg_flange_base_fixed_joint: type fixed, parent qbhand1_base_link, child qbhand1_90_deg_flange_base_link, origin xyz=0 0 0 rpy=-1.57 0 0
- added joint qbhand1_base_fixed_joint: type fixed, parent panda_link8, child qbhand1_base_link, origin xyz=0.045 0 0.035 rpy=1.57 0 1.57
- added joint qbhand1_index_distal_joint: type revolute, parent qbhand1_index_middle_link, child qbhand1_index_distal_virtual_link, origin xyz=0.009 0 0 rpy=0 0 0, axis 0 0 -1, limit lower=0.0 upper=0.785 effort=100 velocity=100, mimic joint=qbhand1_synergy_joint multiplier=0.785
- added joint qbhand1_index_distal_virtual_joint: type revolute, parent qbhand1_index_distal_virtual_link, child qbhand1_index_distal_link, origin xyz=0.013 0 0 rpy=0 0 0, axis 0 0 -1, limit lower=0.0 upper=0.785 effort=100 velocity=100, mimic joint=qbhand1_index_distal_joint multiplier=1.0
- added joint qbhand1_index_knuckle_joint: type revolute, parent qbhand1_palm_link, child qbhand1_index_knuckle_link, origin xyz=-0.02 -0.007 0.014 rpy=0 0 1.57, axis 0 0 -1, limit lower=-0.524 upper=0.524 effort=100 velocity=100, mimic joint=qbhand1_synergy_joint multiplier=-0.2
- added joint qbhand1_index_middle_joint: type revolute, parent qbhand1_index_proximal_link, child qbhand1_index_middle_virtual_link, origin xyz=0.017 0 0 rpy=0 0 0, axis 0 0 -1, limit lower=0.0 upper=0.785 effort=100 velocity=100, mimic joint=qbhand1_synergy_joint multiplier=0.785
- added joint qbhand1_index_middle_virtual_joint: type revolute, parent qbhand1_index_middle_virtual_link, child qbhand1_index_middle_link, origin xyz=0.013 0 0 rpy=0 0 0, axis 0 0 -1, limit lower=0.0 upper=0.785 effort=100 velocity=100, mimic joint=qbhand1_index_middle_joint multiplier=1.0
- added joint qbhand1_index_proximal_joint: type revolute, parent qbhand1_index_knuckle_link, child qbhand1_index_proximal_virtual_link, origin xyz=0.009 0 0 rpy=1.57 0 0, axis 0 0 -1, limit lower=0.0 upper=0.785 effort=100 velocity=100, mimic joint=qbhand1_synergy_joint multiplier=0.785
- added joint qbhand1_index_proximal_virtual_joint: type revolute, parent qbhand1_index_proximal_virtual_link, child qbhand1_index_proximal_link, origin xyz=0.013 0 0 rpy=0 0 0, axis 0 0 -1, limit lower=0.0 upper=0.785 effort=100 velocity=100, mimic joint=qbhand1_index_proximal_joint multiplier=1.0
- added joint qbhand1_little_distal_joint: type revolute, parent qbhand1_little_middle_link, child qbhand1_little_distal_virtual_link, origin xyz=0.009 0 0 rpy=0 0 0, axis 0 0 -1, limit lower=0.0 upper=0.785 effort=100 velocity=100, mimic joint=qbhand1_synergy_joint multiplier=0.785
- added joint qbhand1_little_distal_virtual_joint: type revolute, parent qbhand1_little_distal_virtual_link, child qbhand1_little_distal_link, origin xyz=0.013 0 0 rpy=0 0 0, axis 0 0 -1, limit lower=0.0 upper=0.785 effort=100 velocity=100, mimic joint=qbhand1_little_distal_joint multiplier=1.0
- added joint qbhand1_little_knuckle_joint: type revolute, parent qbhand1_palm_link, child qbhand1_little_knuckle_link, origin xyz=0.04 -0.012 0.014 rpy=0 0 1.57, axis 0 0 -1, limit lower=-0.524 upper=0.524 effort=100 velocity=100, mimic joint=qbhand1_synergy_joint multiplier=0.4
- added joint qbhand1_little_middle_joint: type revolute, parent qbhand1_little_proximal_link, child qbhand1_little_middle_virtual_link, origin xyz=0.009 0 0 rpy=0 0 0, axis 0 0 -1, limit lower=0.0 upper=0.785 effort=100 velocity=100, mimic joint=qbhand1_synergy_joint multiplier=0.785
- added joint qbhand1_little_middle_virtual_joint: type revolute, parent qbhand1_little_middle_virtual_link, child qbhand1_little_middle_link, origin xyz=0.013 0 0 rpy=0 0 0, axis 0 0 -1, limit lower=0.0 upper=0.785 effort=100 velocity=100, mimic joint=qbhand1_little_middle_joint multiplier=1.0
- added joint qbhand1_little_proximal_joint: type revolute, parent qbhand1_little_knuckle_link, child qbhand1_little_proximal_virtual_link, origin xyz=0.009 0 0 rpy=1.57 0 0, axis 0 0 -1, limit lower=0.0 upper=0.785 effort=100 velocity=100, mimic joint=qbhand1_synergy_joint multiplier=0.785
- added joint qbhand1_little_proximal_virtual_joint: type revolute, parent qbhand1_little_proximal_virtual_link, child qbhand1_little_proximal_link, origin xyz=0.013 0 0 rpy=0 0 0, axis 0 0 -1, limit lower=0.0 upper=0.785 effort=100 velocity=100, mimic joint=qbhand1_little_proximal_joint multiplier=1.0
- added joint qbhand1_middle_distal_joint: type revolute, parent qbhand1_middle_middle_link, child qbhand1_middle_distal_virtual_link, origin xyz=0.009 0 0 rpy=0 0 0, axis 0 0 -1, limit lower=0.0 upper=0.785 effort=100 velocity=100, mimic joint=qbhand1_synergy_joint multiplier=0.785
- added joint qbhand1_middle_distal_virtual_joint: type revolute, parent qbhand1_middle_distal_virtual_link, child qbhand1_middle_distal_link, origin xyz=0.013 0 0 rpy=0 0 0, axis 0 0 -1, limit lower=0.0 upper=0.785 effort=100 velocity=100, mimic joint=qbhand1_middle_distal_joint multiplier=1.0
- added joint qbhand1_middle_knuckle_joint: type revolute, parent qbhand1_palm_link, child qbhand1_middle_knuckle_link, origin xyz=0 0 0.014 rpy=0 0 1.57, axis 0 0 -1, limit lower=-0.524 upper=0.524 effort=100 velocity=100, mimic joint=qbhand1_synergy_joint multiplier=0.0
- added joint qbhand1_middle_middle_joint: type revolute, parent qbhand1_middle_proximal_link, child qbhand1_middle_middle_virtual_link, origin xyz=0.017 0 0 rpy=0 0 0, axis 0 0 -1, limit lower=0.0 upper=0.785 effort=100 velocity=100, mimic joint=qbhand1_synergy_joint multiplier=0.785
- added joint qbhand1_middle_middle_virtual_joint: type revolute, parent qbhand1_middle_middle_virtual_link, child qbhand1_middle_middle_link, origin xyz=0.013 0 0 rpy=0 0 0, axis 0 0 -1, limit lower=0.0 upper=0.785 effort=100 velocity=100, mimic joint=qbhand1_middle_middle_joint multiplier=1.0
- added joint qbhand1_middle_proximal_joint: type revolute, parent qbhand1_middle_knuckle_link, child qbhand1_middle_proximal_virtual_link, origin xyz=0.009 0 0 rpy=1.57 0 0, axis 0 0 -1, limit lower=0.0 upper=0.785 effort=100 velocity=100, mimic joint=qbhand1_synergy_joint multiplier=0.785
- added joint qbhand1_middle_proximal_virtual_joint: type revolute, parent qbhand1_middle_proximal_virtual_link, child qbhand1_middle_proximal_link, origin xyz=0.013 0 0 rpy=0 0 0, axis 0 0 -1, limit lower=0.0 upper=0.785 effort=100 velocity=100, mimic joint=qbhand1_middle_proximal_joint multiplier=1.0
- added joint qbhand1_palm_fixed_joint: type fixed, parent qbhand1_base_link, child qbhand1_palm_link, origin xyz=-0.0045 0.0145 0.144 rpy=1.57 0 0
- added joint qbhand1_ring_distal_joint: type revolute, parent qbhand1_ring_middle_link, child qbhand1_ring_distal_virtual_link, origin xyz=0.009 0 0 rpy=0 0 0, axis 0 0 -1, limit lower=0.0 upper=0.785 effort=100 velocity=100, mimic joint=qbhand1_synergy_joint multiplier=0.785
- added joint qbhand1_ring_distal_virtual_joint: type revolute, parent qbhand1_ring_distal_virtual_link, child qbhand1_ring_distal_link, origin xyz=0.013 0 0 rpy=0 0 0, axis 0 0 -1, limit lower=0.0 upper=0.785 effort=100 velocity=100, mimic joint=qbhand1_ring_distal_joint multiplier=1.0
- added joint qbhand1_ring_knuckle_joint: type revolute, parent qbhand1_palm_link, child qbhand1_ring_knuckle_link, origin xyz=0.02 -0.007 0.014 rpy=0 0 1.57, axis 0 0 -1, limit lower=-0.524 upper=0.524 effort=100 velocity=100, mimic joint=qbhand1_synergy_joint multiplier=0.2
- added joint qbhand1_ring_middle_joint: type revolute, parent qbhand1_ring_proximal_link, child qbhand1_ring_middle_virtual_link, origin xyz=0.017 0 0 rpy=0 0 0, axis 0 0 -1, limit lower=0.0 upper=0.785 effort=100 velocity=100, mimic joint=qbhand1_synergy_joint multiplier=0.785
- added joint qbhand1_ring_middle_virtual_joint: type revolute, parent qbhand1_ring_middle_virtual_link, child qbhand1_ring_middle_link, origin xyz=0.013 0 0 rpy=0 0 0, axis 0 0 -1, limit lower=0.0 upper=0.785 effort=100 velocity=100, mimic joint=qbhand1_ring_middle_joint multiplier=1.0
- added joint qbhand1_ring_proximal_joint: type revolute, parent qbhand1_ring_knuckle_link, child qbhand1_ring_proximal_virtual_link, origin xyz=0.009 0 0 rpy=1.57 0 0, axis 0 0 -1, limit lower=0.0 upper=0.785 effort=100 velocity=100, mimic joint=qbhand1_synergy_joint multiplier=0.785
- added joint qbhand1_ring_proximal_virtual_joint: type revolute, parent qbhand1_ring_proximal_virtual_link, child qbhand1_ring_proximal_link, origin xyz=0.013 0 0 rpy=0 0 0, axis 0 0 -1, limit lower=0.0 upper=0.785 effort=100 velocity=100, mimic joint=qbhand1_ring_proximal_joint multiplier=1.0
- added joint qbhand1_synergy_joint: type revolute, parent qbhand1_palm_link, child qbhand1_synergy_tendon_virtual_link, origin xyz=0 0 0 rpy=0 0 0, axis 0 0 1, limit lower=0.0 upper=1.0 effort=100 velocity=100
- added joint qbhand1_thumb_distal_joint: type revolute, parent qbhand1_thumb_proximal_link, child qbhand1_thumb_distal_virtual_link, origin xyz=0.009 0 0 rpy=0 0 0, axis 0 0 -1, limit lower=0.0 upper=0.785 effort=100 velocity=100, mimic joint=qbhand1_synergy_joint multiplier=0.785
- added joint qbhand1_thumb_distal_virtual_joint: type revolute, parent qbhand1_thumb_distal_virtual_link, child qbhand1_thumb_distal_link, origin xyz=0.013 0 0 rpy=0 0 0, axis 0 0 -1, limit lower=0.0 upper=0.785 effort=100 velocity=100, mimic joint=qbhand1_thumb_distal_joint multiplier=1.0
- added joint qbhand1_thumb_knuckle_joint: type revolute, parent qbhand1_palm_link, child qbhand1_thumb_knuckle_link, origin xyz=-0.044 -0.0465 -0.002 rpy=-1.57 3.14 0.0, axis 0 0 -1, limit lower=0.0 upper=1.571 effort=100 velocity=100, mimic joint=qbhand1_synergy_joint multiplier=2.542
- added joint qbhand1_thumb_proximal_joint: type revolute, parent qbhand1_thumb_knuckle_link, child qbhand1_thumb_proximal_virtual_link, origin xyz=0.0255 -0.0038 -0.00012 rpy=-1.1415 0.0 0.0, axis 0 0 -1, limit lower=0.0 upper=0.785 effort=100 velocity=100, mimic joint=qbhand1_synergy_joint multiplier=0.785
- added joint qbhand1_thumb_proximal_virtual_joint: type revolute, parent qbhand1_thumb_proximal_virtual_link, child qbhand1_thumb_proximal_link, origin xyz=0.013 0 0 rpy=0 0 0, axis 0 0 -1, limit lower=0.0 upper=0.785 effort=100 velocity=100, mimic joint=qbhand1_thumb_proximal_joint multiplier=1.0
- added joint thumb_index_ee_joint: type fixed, parent right_hand_ee_link, child thumb_index_ee_link, origin xyz=0.07 -0.04 0.03 rpy=0 0.5 -1.0
- joint panda_joint: origin xyz=-0.18 0.0 0.47 rpy=0.0 0.0 0.0 -> xyz=0.12 0.0 0.47 rpy=0.0 0.0 0.0
- joint right_hand_ee_joint: origin xyz=0.102 -0.003 0.037 rpy=0 0 0 -> xyz=0.13 -0.003 0.037 rpy=0 0 0
